File: UnifiedBreakout/UnifiedBreakout/argon_estop.sch (KiCad schematic (older format))
At the start: 1 part, among them J15 ARGON J2.2

Commit message: More placement, add some custom parts
Parts:
- J15: footprint Connector_RJ:RJ45_Ninigi_GE -> Stewart:SS6488SANF1
Changed lines of the file:
@@
 F 0 "J15" H 5220 3404 50  0000 R CNN
 F 1 "ARGON J2.2" H 5220 3495 50  0000 R CNN
-F 2 "Connector_RJ:RJ45_Ninigi_GE" V 5550 3425 50  0001 C CNN
+F 2 "Stewart:SS6488SANF1" V 5550 3425 50  0001 C CNN
 F 3 "~" V 5550 3425 50  0001 C CNN
 	1    5550 3400

Commit message: Assigned some parts
Parts:
- J15: MPN (none) -> SS-6488S-A-NF-1; Manufacturer (none) -> Bel
Changed lines of the file:
@@
 F 2 "Stewart:SS6488SANF1" V 5550 3425 50  0001 C CNN
 F 3 "~" V 5550 3425 50  0001 C CNN
+F 4 "SS-6488S-A-NF-1" H 5550 3400 50  0001 C CNN "MPN"
+F 5 "Bel" H 5550 3400 50  0001 C CNN "Manufacturer"
 	1    5550 3400
 	-1   0    0    1
