File: UnifiedBreakout/UnifiedBreakout/UnifiedBreakout.kicad_pcb (KiCad board)
At the start: 2 copper layers, 239.4 x 216.5 mm, 94 parts, among them J1 24V DC IN, J10 MESA P2 INTERNAL IO, J11 MESA P3 REAR IO, J12 ENCODER IN, J13 ENCODER OUT, J14 ARGON J5, J15 ARGON J2.2, J16 RJ14, J17 RJ14, J18 RJ14, J19 RJ14, J2 ATX-24, J20 RJ14, J21 PENDANT, J22 DRAWBAR, J23 MIST, J24 AXIS PWR IN, J25 AXIS PWR OUT, J3 5V BUS, J4 24V BUS, J5 12V BUS, J6 ARGON RS485, J7 RJ45, J8 RJ45, J9 RJ45, Q1 BC547, Q2 BC547, Q3 BC547, U1 4N35, U2 4N35, U3 4N35, U4 4N35, U5 4N35, U6 4N35, U7 74HC14

Commit message: Finished(?) unified breakout layout
Parts:
- removed J6: ARGON RS485, Connector_Phoenix_MSTB:PhoenixContact_MSTBA_2,5_3-G-5,08_1x03_P5.08mm_Horizontal
- added H5: MountingHole, MountingHole:MountingHole_3.2mm_M3, F.Cu at (189.2, 128.3)
- added H6: MountingHole, MountingHole:MountingHole_3.2mm_M3, F.Cu at (264.2, 171.4)
- D5: value LED -> AXIS PWR
- D7: value LED -> DRAWBAR
- D9: value LED -> MIST
- moved J24 200.6 mm to (233.2, 218.7), turned to 0 degrees
- moved J25 197.8 mm to (208.8, 218.7), turned to 0 degrees
- moved J15 176.2 mm to (209.6, 123.2)
- moved U1 174.4 mm to (200.2, 136.9)
- moved R6 173.3 mm to (212.1, 137.2), turned to 270 degrees
- moved J7 163.7 mm to (147.3, 123.2), turned to 180 degrees
- moved R4 146.3 mm to (265.4, 146.1), turned to 90 degrees
- moved R5 140.3 mm to (261.6, 135.9), turned to 270 degrees
- moved J8 136.1 mm to (126.4, 123.2), turned to 180 degrees
- moved R1 132.1 mm to (265.4, 133.3), turned to 90 degrees
- moved D9 127.3 mm to (232.4, 160.0), turned to 180 degrees
- moved J23 123.6 mm to (228.9, 115.6)
- moved D10 122.9 mm to (231.1, 153.7)
- moved RL3 122.5 mm to (229.9, 148.6)
- moved JP3 121.6 mm to (166.4, 133.3), turned to 270 degrees
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Connections:
- J12 pad 10: Net-(J12-Pad10) -> GND
- J16 pad 3: Net-(J16-Pad3) -> GND
- J16 pad 4: GND -> Net-(J16-Pad4)
- J17 pad 3: Net-(J17-Pad3) -> GND
- J17 pad 4: GND -> Net-(J17-Pad4)
- J18 pad 3: Net-(J18-Pad3) -> GND
- J18 pad 4: GND -> Net-(J18-Pad4)
- J19 pad 3: Net-(J19-Pad3) -> GND
- J19 pad 4: GND -> Net-(J19-Pad4)
- J20 pad 3: Net-(J20-Pad3) -> GND
- J20 pad 4: GND -> Net-(J20-Pad4)
- J7 pad 1: /MESA P3 REAR IO/IO_02_STEPGEN_00_STEP -> GND
- J7 pad 2: GND -> /MESA P3 REAR IO/IO_02_STEPGEN_00_STEP
- J7 pad 3: /X MOT/DIR -> GND
- J7 pad 4: GND -> /X MOT/DIR
- J7 pad 5: /X MOT/ENABLE -> GND
- J7 pad 6: GND -> /X MOT/ENABLE
- J7 pad 7: /ALARM -> GND
- J7 pad 8: GND -> /ALARM
- J8 pad 1: /MESA P3 REAR IO/IO_06_STEPGEN_01_STEP -> GND
- J8 pad 2: GND -> /MESA P3 REAR IO/IO_06_STEPGEN_01_STEP
- J8 pad 3: /Y MOT/DIR -> GND
- J8 pad 4: GND -> /Y MOT/DIR
- J8 pad 5: /Y MOT/ENABLE -> GND
- J8 pad 6: GND -> /Y MOT/ENABLE
- J8 pad 7: /ALARM -> GND
- J8 pad 8: GND -> /ALARM
- J9 pad 1: /MESA P3 REAR IO/IO_09_STEPGEN_02_STEP -> GND
- J9 pad 2: GND -> /MESA P3 REAR IO/IO_09_STEPGEN_02_STEP
- J9 pad 3: /Z MOT/DIR -> GND
- J9 pad 4: GND -> /Z MOT/DIR
- J9 pad 5: /Z MOT/ENABLE -> GND
- J9 pad 6: GND -> /Z MOT/ENABLE
- J9 pad 7: /ALARM -> GND
- J9 pad 8: GND -> /ALARM
- U2 pad 1: Net-(J16-Pad3) -> Net-(J16-Pad4)
- U3 pad 1: Net-(J17-Pad3) -> Net-(J17-Pad4)
- U4 pad 1: Net-(J18-Pad3) -> Net-(J18-Pad4)
- U5 pad 1: Net-(J19-Pad3) -> Net-(J19-Pad4)
- U6 pad 1: Net-(J20-Pad3) -> Net-(J20-Pad4)
- U7 pad 14: (no net) -> +5VP
- U7 pad 7: (no net) -> GND
Routing:
- net +24V: track 0.00 -> 700.3 mm, vias 0 -> 2
- net +5V: track 0.00 -> 511.8 mm
- net +5VP: track 0.00 -> 370.2 mm
- net +12V: track 0.00 -> 308.9 mm
- net /ATX_PWR: track 0.00 -> 230.4 mm, vias 0 -> 4
- net /ESTOP: track 0.00 -> 226.8 mm, vias 0 -> 2
- net /SPINDLE_STEPGEN_DIR: track 0.00 -> 207.6 mm
- net /SPINDLE_STEPGEN_STEP: track 0.00 -> 206.6 mm
- net /SPINDLE_PWM_DIR: track 0.00 -> 203.4 mm
- net /ALARM: track 0.00 -> 198.4 mm
- net /SPINDLE_PWM_SIG: track 0.00 -> 191.2 mm
- net /X MOT/DIR: track 0.00 -> 177.5 mm
- net /MESA P3 REAR IO/IO_02_STEPGEN_00_STEP: track 0.00 -> 177.4 mm
- net /SPINDLE_ENC_IDX: track 0.00 -> 163.2 mm
- net /Y MOT/DIR: track 0.00 -> 162.4 mm
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- added copper zone on B.Cu, net GND
- added copper zone on F.Cu, net GND
Other:
- board size 239.4 x 216.5 mm -> 307.3 x 121.9 mm
- net class Default: clearance 0.2 -> 0.15; trace_width 0.35 -> 0.3
- net class ESTOP added: clearance 0.15, trace_width 0.35, via_dia 1, via_drill 0.7
- net class High power: clearance 0.5 -> 0.6; via_dia 0.8 -> 1.5; via_drill 0.4 -> 1
- net class Low power: via_dia 0.8 -> 1; via_drill 0.4 -> 0.7
- net class Mains: clearance 2.5 -> 1.75; via_dia 0.8 -> 3; via_drill 0.4 -> 1.5
- rule trace_clearance: 0.2 -> 0.15
- board text added: "+"
