File: UnifiedBreakout/UnifiedBreakout/UnifiedBreakout.kicad_pcb (KiCad board)
At the start: 2 copper layers, 200 x 100 mm, 68 parts, among them J1 DRAWBAR+MIST, J14 ARGON J5, J15 ARGON J2.2, J2 Screw_Terminal_01x05, J21 PENDANT, J24 AXIS PWR IN, J25 AXIS PWR OUT, J3 Dual DA15 Stacked, J4 24V BUS, J5 DB25_Receptacle_Dual, J7 RJ45, J8 RJ45, J9 RJ45, Q1 BC547, Q2 2N7000, Q4 2N7000, U1 4N35, U2 4N35, U3 4N35, U4 4N35, U5 4N35, U6 4N35, U7 74HC14, U9 4N35

Commit message: Grouped 4 way RJ45s
Parts:
- removed J15: ARGON J2.2, Stewart:SS6488SANF1
- removed J7, J9: RJ45, Stewart:SS6488SANF1
- J8: value RJ45 -> ~; footprint Stewart:SS6488SANF1 -> UnifiedBreakout:SS71800-041F
- moved J2 138.3 mm to (-53.3, 63.5), turned to -90 degrees
- moved J8 134.6 mm to (139.7, 16.5)
- moved J14 70.2 mm to (83.8, 20.3), turned to -90 degrees

Commit message: Update IO and opto
Parts:
- removed C7: 100n, Capacitor_THT:C_Disc_D5.0mm_W2.5mm_P5.00mm
- removed C8: 100uF, Capacitor_THT:CP_Radial_D8.0mm_P3.50mm
- removed D5: LED, LED_THT:LED_D3.0mm
- removed D6: 1N4001, Diode_THT:D_DO-41_SOD81_P10.16mm_Horizontal
- removed H5, H6: MountingHole, MountingHole:MountingHole_3.2mm_M3
- removed J14: ARGON J5, Connector_IDC:IDC-Header_2x13_P2.54mm_Vertical
- removed J21: PENDANT, Connector_Dsub:DSUB-25_Female_Horizontal_P2.77x2.84mm_EdgePinOffset7.70mm_Housed_MountingHolesOffset9.12mm
- removed J24: AXIS PWR IN, Connector_Phoenix_MSTB:PhoenixContact_MSTBA_2,5_3-G-5,08_1x03_P5.08mm_Horizontal
- removed J25: AXIS PWR OUT, Connector_Phoenix_MSTB:PhoenixContact_MSTBA_2,5_3-G-5,08_1x03_P5.08mm_Horizontal
- removed JP3: HSIN2, Connector_PinHeader_2.54mm:PinHeader_1x03_P2.54mm_Vertical
- removed Q1: BC547, Package_TO_SOT_THT:TO-92_Inline
- removed Q2, Q4: 2N7000, Package_TO_SOT_THT:TO-92_Inline
- removed R14, R8: 2K2, Resistor_THT:R_Axial_DIN0207_L6.3mm_D2.5mm_P7.62mm_Horizontal
- removed R2: 220R, Resistor_THT:R_Axial_DIN0207_L6.3mm_D2.5mm_P7.62mm_Horizontal
- removed R24, R26, R27, R28, R29, R30, R31: 10K, Resistor_THT:R_Axial_DIN0207_L6.3mm_D2.5mm_P7.62mm_Horizontal
- removed R5: 220K, Resistor_THT:R_Axial_DIN0207_L6.3mm_D2.5mm_P7.62mm_Horizontal
- removed RL1: JW2, Relay_THT:Relay_DPDT_Panasonic_JW2
- removed U1, U2, U3, U4, U5: 4N35, Package_DIP:DIP-6_W7.62mm
- added C1: 100n, Capacitor_THT:C_Disc_D5.0mm_W2.5mm_P5.00mm, F.Cu at (182.9, 55.9)
- added C2: 100uF, Capacitor_THT:CP_Radial_D8.0mm_P3.50mm, F.Cu at (181.3, 45.7)
- added J6: DRAWBAR+MIST+AXIS_PWR, Connector_Phoenix_MSTB:PhoenixContact_MSTBA_2,5_3-G-5,08_1x03_P5.08mm_Horizontal, F.Cu at (50.8, 34.3)
- added J7: LIMIT, Connector_Phoenix_MSTB:PhoenixContact_MSTBA_2,5_3-G-5,08_1x03_P5.08mm_Horizontal, F.Cu at (172.7, 141.0)
- added J9: AUX, Connector_Phoenix_MSTB:PhoenixContact_MSTBA_2,5_3-G-5,08_1x03_P5.08mm_Horizontal, F.Cu at (154.9, 139.7)
- added JP1: HSIN1, Connector_PinHeader_2.54mm:PinHeader_1x03_P2.54mm_Vertical, F.Cu at (37.1, 64.3)
- added R12: 10K, Resistor_THT:R_Axial_DIN0207_L6.3mm_D2.5mm_P7.62mm_Horizontal, F.Cu at (86.4, 110.7)
- added R13: 2K2, Resistor_THT:R_Axial_DIN0207_L6.3mm_D2.5mm_P7.62mm_Horizontal, F.Cu at (135.9, 81.3)
- added R25: 10K, Resistor_THT:R_Axial_DIN0207_L6.3mm_D2.5mm_P7.62mm_Horizontal, F.Cu at (115.6, 113.3)
- added U11: ILD74, Package_DIP:DIP-8_W7.62mm_LongPads, F.Cu at (183.6, 87.8)
- added U12: ILD74, Package_DIP:DIP-8_W7.62mm_LongPads, F.Cu at (197.2, 101.6)
- added U13: ILD74, Package_DIP:DIP-8_W7.62mm_LongPads, F.Cu at (210.8, 87.8)
- added U8: G3VM-61A1, Package_DIP:DIP-4_W7.62mm, F.Cu at (34.3, 52.1)
- J1: value DRAWBAR+MIST -> Dual DA15 Stacked; footprint Connector_Phoenix_MSTB:PhoenixContact_MSTBA_2,5_2-G-5,08_1x02_P5.08mm_Horizontal -> UnifiedBreakout:NorComp-Dual-DA15
- J2: value Screw_Terminal_01x05 -> ARGON J5; footprint Connector_Phoenix_MSTB:PhoenixContact_MSTBA_2,5_6-G-5,08_1x06_P5.08mm_Horizontal -> Connector_IDC:IDC-Header_2x13_P2.54mm_Vertical
- J3: value Dual DA15 Stacked -> ~; footprint UnifiedBreakout:NorComp-Dual-DA15 -> UnifiedBreakout:SS71800-041F
- J4: value 24V BUS -> PENDANT; footprint Connector_Phoenix_MSTB:PhoenixContact_MSTBA_2,5_2-G-5,08_1x02_P5.08mm_Horizontal -> Connector_Dsub:DSUB-25_Female_Horizontal_P2.77x2.84mm_EdgePinOffset7.70mm_Housed_MountingHolesOffset9.12mm
- J5: value DB25_Receptacle_Dual -> 24V BUS; footprint UnifiedBreakout:NorComp-Dual-DB25 -> Connector_Phoenix_MSTB:PhoenixContact_MSTBA_2,5_2-G-5,08_1x02_P5.08mm_Horizontal
- J8: value ~ -> DB25_Receptacle_Dual; footprint UnifiedBreakout:SS71800-041F -> UnifiedBreakout:NorComp-Dual-DB25
- JP2: value HSIN1 -> HSIN2
- R1, R10: value 10K -> 2K2
- R15, R6: value 220K -> 10K
- R16: value 2K2 -> 220R
- R17: value 220K -> 220R
- R19, R23: value 220K -> 2K2
- R3: value 220R -> 10K
- R9: value 680R -> 10K
- U6: value 4N35 -> G3VM-61A1; footprint Package_DIP:DIP-6_W7.62mm -> Package_DIP:DIP-4_W7.62mm
- U7: value 74HC14 -> G3VM-61A1; footprint Package_DIP:DIP-14_W7.62mm_LongPads -> Package_DIP:DIP-4_W7.62mm
- moved J5 217.0 mm to (182.9, 33.0), turned to 180 degrees
- moved J2 190.7 mm to (137.2, 55.9)
- moved H4 158.8 mm to (193.0, 144.8)
- moved H2 150.6 mm to (193.0, 27.9)
- moved J3 131.2 mm to (132.1, 34.3)
- moved J8 130.8 mm to (79.4, 132.7), turned to 0 degrees
- moved J1 130.7 mm to (69.0, 34.8), turned to 180 degrees
- moved U6 103.7 mm to (52.1, 52.1), turned to 90 degrees
- moved H3 90.4 mm to (30.5, 144.8)
- moved R1 67.3 mm to (128.3, 106.7)
- moved R3 67.3 mm to (128.3, 114.8)
- moved R6 67.3 mm to (128.3, 118.8)
- moved R7 67.3 mm to (128.3, 122.9)
- moved D2 66.0 mm to (45.7, 124.5)
- moved J4 65.4 mm to (136.0, 139.9), turned to 0 degrees
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Connections:
- C3 pad 1: +24V -> +5VP
- C4 pad 1: +24V -> +5VP
- J2 pad 1: /LIM X/INPUT -> GND
- J2 pad 2: /LIM Y/INPUT -> unconnected-(J2-Pin_2-Pad2)
- J2 pad 3: /LIM Z/INPUT -> unconnected-(J2-Pin_3-Pad3)
- J2 pad 4: /PROBE/INPUT -> Net-(J2-Pin_4)
- J2 pad 5: /TOOL_PROBE/INPUT -> unconnected-(J2-Pin_5-Pad5)
- J2 pad 6: /DRAWBAR SW/INPUT -> Net-(J2-Pin_6)
- J4 pad 1: +24V -> /PENDANT_SELX
- J4 pad 2: GND -> /PENDANT_SELZ
- JP2 pad 1: /SPINDLE_PWM_DIR -> /SPINDLE_PWM_SIG
- JP2 pad 2: Net-(J14-Pin_4) -> Net-(J2-Pin_6)
- JP2 pad 3: /SPINDLE_STEPGEN_STEP -> /SPINDLE_STEPGEN_DIR
- R1 pad 1: +5VP -> Net-(R1-Pad1)
- R1 pad 2: /DRAWBAR_VALVE -> GND
- R10 pad 1: +5VP -> Net-(R10-Pad1)
- R10 pad 2: /TOOL_PROBE -> GND
- R15 pad 1: Net-(R15-Pad1) -> +5VP
- R15 pad 2: GND -> /LIMIT_Y
- R16 pad 1: Net-(R16-Pad1) -> Net-(D1-A)
- R16 pad 2: GND -> +5VP
- R17 pad 1: Net-(R17-Pad1) -> /MESA P2 INTERNAL IO/MESA_5V
- R17 pad 2: GND -> Net-(D2-A)
- R18 pad 1: Net-(R18-Pad1) -> +5VP
- R18 pad 2: GND -> Net-(R18-Pad2)
- R19 pad 1: Net-(R19-Pad1) -> +5VP
- R19 pad 2: GND -> Net-(R19-Pad2)
- R20 pad 1: Net-(R20-Pad1) -> +5VP
- R20 pad 2: GND -> Net-(R20-Pad2)
- R3 pad 1: /MESA P2 INTERNAL IO/MESA_5V -> +5VP
- R3 pad 2: Net-(D2-A) -> /LIMIT_X
- R6 pad 1: Net-(R6-Pad1) -> +5VP
- R6 pad 2: GND -> /DRAWBAR_SW
- R9 pad 1: Net-(D5-K) -> +5VP
- R9 pad 2: Net-(D6-A) -> /PROBE
- U6 pad 1: /DRAWBAR SW/INPUT -> Net-(R18-Pad2)
- U6 pad 2: Net-(R22-Pad1) -> /DRAWBAR_VALVE
- U6 pad 3: unconnected-(U6-NC-Pad3) -> GND
- U6 pad 4: GND -> Net-(J6-Pin_1)
- U7 pad 1: /AXIS_PWR -> Net-(R19-Pad2)
- U7 pad 2: /AXIS POWER RELAY/ENABLE -> /MIST
- U7 pad 3: /DRAWBAR_VALVE -> GND
- U9 pad 1: /TOOL_PROBE/INPUT -> /ARGON ESTOP/ESTOP+
- U9 pad 2: Net-(R4-Pad1) -> Net-(R22-Pad1)
- U9 pad 5: /TOOL_PROBE -> /ESTOP
- U9 pad 6: Net-(R5-Pad1) -> Net-(R21-Pad1)
Other:
- board size 200 x 100 mm -> 172.7 x 127.1 mm

Commit message: Tweaks and stuff
Parts:
- added D3: +24V, LED_THT:LED_D3.0mm, F.Cu at (155.0, 75.9)
- added R2: 220R, Resistor_THT:R_Axial_DIN0207_L6.3mm_D2.5mm_P7.62mm_Horizontal, F.Cu at (154.9, 71.1)
- moved U11 34.3 mm to (149.9, 94.0)
- moved U13 33.4 mm to (180.3, 101.6), turned to 90 degrees
- moved U12 25.7 mm to (172.7, 94.0), turned to -90 degrees
- moved H4 17.0 mm to (185.4, 160.0)
- moved J3 17.0 mm to (124.5, 49.5)
- moved J4 17.0 mm to (128.4, 155.1)
- moved J7 17.0 mm to (165.1, 156.2)
- moved J9 17.0 mm to (147.3, 154.9)
- moved R16 17.0 mm to (164.9, 133.1)
- moved R3 17.0 mm to (120.7, 130.0)
- moved R7 17.0 mm to (120.7, 138.1)
- moved U9 17.0 mm to (102.9, 139.7)
- moved H3 17.0 mm to (22.9, 160.0)
- moved U7 17.0 mm to (35.6, 66.0)
- moved C1 17.0 mm to (175.3, 71.1)
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
Commit message: Started some layout
Parts:
- removed J1: Dual DA15 Stacked, UnifiedBreakout:NorComp-Dual-DA15
- added H5: MountingHole, MountingHole:MountingHole_3.2mm_M3, F.Cu at (97.8, 43.2)
- added H6: MountingHole, MountingHole:MountingHole_3.2mm_M3, F.Cu at (172.7, 158.8)
- added J10: DA15_Receptacle_MountingHoles, Connector_Dsub:DSUB-15_Female_Vertical_P2.77x2.84mm_MountingHoles, F.Cu at (71.8, 77.5)
- added J11: DA15_Receptacle_MountingHoles, Connector_Dsub:DSUB-15_Female_Vertical_P2.77x2.84mm_MountingHoles, F.Cu at (71.8, 92.6)
- moved R17 132.2 mm to (33.0, 128.3), turned to -90 degrees
- moved R16 128.2 mm to (36.8, 135.9), turned to 90 degrees
- moved J7 118.3 mm to (116.8, 48.3), turned to 180 degrees
- moved U8 118.1 mm to (144.8, 68.6)
- moved U7 115.6 mm to (151.1, 68.6)
- moved U6 113.0 mm to (157.5, 68.6)
- moved J6 113.0 mm to (156.2, 48.3)
- moved J9 107.4 mm to (134.6, 48.3), turned to 180 degrees
- moved H4 83.5 mm to (102.9, 147.3)
- moved JP1 79.8 mm to (109.2, 82.5), turned to 90 degrees
- moved R19 64.2 mm to (151.1, 78.7), turned to 90 degrees
- moved J3 62.2 mm to (62.2, 49.5)
- moved R18 58.0 mm to (157.5, 78.7), turned to 90 degrees
- moved R20 35.5 mm to (144.8, 78.7), turned to 90 degrees
- moved H1 28.4 mm to (35.6, 68.6)
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Connections:
- J3 pad 1_1: GND -> +24V
- J3 pad 1_4: +24V -> GND
- J3 pad 2_1: /MESA P3 REAR IO/IO_02_STEPGEN_00_STEP -> unconnected-(J3A-P2_1-Pad2_1)
- J3 pad 2_2: /MESA P3 REAR IO/IO_06_STEPGEN_01_STEP -> /MESA P3 REAR IO/IO_09_STEPGEN_02_STEP
- J3 pad 2_3: /MESA P3 REAR IO/IO_09_STEPGEN_02_STEP -> /MESA P3 REAR IO/IO_06_STEPGEN_01_STEP
- J3 pad 2_4: unconnected-(J3D-P2_4-Pad2_4) -> /MESA P3 REAR IO/IO_02_STEPGEN_00_STEP
- J3 pad 3_1: GND -> /ARGON ESTOP/RS485_A
- J3 pad 3_4: /ARGON ESTOP/RS485_A -> GND
- J3 pad 4_1: /MESA P3 REAR IO/IO_04_STEPGEN_00_DIR -> /ARGON ESTOP/ESTOP+
- J3 pad 4_2: /MESA P3 REAR IO/IO_08_STEPGEN_01_DIR -> /MESA P3 REAR IO/IO_10_STEPGEN_02_DIR
- J3 pad 4_3: /MESA P3 REAR IO/IO_10_STEPGEN_02_DIR -> /MESA P3 REAR IO/IO_08_STEPGEN_01_DIR
- J3 pad 4_4: /ARGON ESTOP/ESTOP+ -> /MESA P3 REAR IO/IO_04_STEPGEN_00_DIR
- J3 pad 6_1: /X MOT/ENABLE -> /ARGON ESTOP/RS485_B
- J3 pad 6_2: /Y MOT/ENABLE -> /Z MOT/ENABLE
- J3 pad 6_3: /Z MOT/ENABLE -> /Y MOT/ENABLE
- J3 pad 6_4: /ARGON ESTOP/RS485_B -> /X MOT/ENABLE
- J3 pad 7_1: GND -> +24V
- J3 pad 7_4: +24V -> GND
- J3 pad 8_1: /ALARM -> GND
- J3 pad 8_4: GND -> /ALARM
- J3 pad S1: GND -> Net-(J3A-SHIELD-PadS1)
- J3 pad S2: GND -> Net-(J3A-SHIELD-PadS1)
- J3 pad S3: GND -> Net-(J3A-SHIELD-PadS1)
- J3 pad S4: GND -> Net-(J3A-SHIELD-PadS1)
- J3 pad S5: GND -> Net-(J3A-SHIELD-PadS1)
- J8 pad MH4: unconnected-(J8-PadMH4) -> GND
Routing:
- net +24V: track 0.00 -> 34.6 mm
- net Net-(J6-Pin_3): track 0.00 -> 13.2 mm
- net Net-(J6-Pin_1): track 0.00 -> 13.2 mm
- net Net-(J6-Pin_2): track 0.00 -> 12.7 mm
- net Net-(D3-A): track 0.00 -> 6.35 mm
Other:
- board size 172.7 x 127.1 mm -> 149.9 x 127.1 mm
- board text added: "+24V"
- board text added: "ARGON J2.2"
- board text added: "ARGON J5"
- board text added: "AXIS PWR"
- board text added: "CNC BREAKOUT V3 J WAPLES MAR 2023"
- board text added: "DB RELEASE"
- board text added: "DRAWBAR"
- board text added: "GND"
- board text added: "LIMIT X"
- board text added: "LIMIT Y"
- board text added: "LIMIT Z"
- board text added: "MIST"
- board text added: "PENDANT"
- board text added: "PROBE"
- board text added: "PWM"
- board text added: "SPINDLE ENCODER"
- board text added: "SPINDLE SOURCE"
- board text added: "STEPGEN"
- board text added: "TOOL SET"
- board text added: "TOP: MESA P3 REAR IO BOTTOM: MESA P2 INTERNAL IO"
- board text added: "X AXIS"
- board text added: "Y AXIS"
- board text added: "Z AXIS"

Commit message: Some layout
Parts:
- removed U13: ILD74, Package_DIP:DIP-8_W7.62mm_LongPads
- added U3: ILD74, Package_DIP:DIP-8_W7.62mm_LongPads, F.Cu at (108.0, 62.2)
- H1, H2, H3, H4, H5, H6: footprint MountingHole:MountingHole_3.2mm_M3 -> MountingHole:MountingHole_3.2mm_M3_Pad
- moved R7 71.0 mm to (100.3, 73.7), turned to -90 degrees
- moved R5 65.7 mm to (133.3, 73.7), turned to -90 degrees
- moved R10 59.4 mm to (87.6, 100.3)
- moved R4 56.0 mm to (87.6, 88.9)
- moved R2 55.8 mm to (87.6, 85.1)
- moved R1 48.7 mm to (114.3, 73.7), turned to -90 degrees
- moved R19 43.5 mm to (128.3, 73.7), turned to -90 degrees
- moved R6 36.6 mm to (87.6, 92.7)
- moved R3 34.5 mm to (119.4, 73.7), turned to -90 degrees
- moved R20 31.8 mm to (87.6, 104.1)
- moved JP1 31.4 mm to (135.9, 99.1)
- moved JP2 31.4 mm to (135.9, 102.9)
- moved R9 31.2 mm to (105.4, 73.7), turned to -90 degrees
- moved R8 30.8 mm to (87.6, 96.5)
- moved U2 30.7 mm to (135.9, 62.2)
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- renumbered J11 to J1, J8 to J10, J10 to J2, J2 to J3, J3 to J4, J4 to J5, J5 to J6, J6 to J7, J7 to J8, R15 to R10, R16 to R11, R17 to R12, R18 to R13, R19 to R14, R20 to R15, R2 to R16, R21 to R17, R22 to R18, R23 to R19, R3 to R2, R25 to R20, R4 to R3, R6 to R4, R7 to R5, R9 to R6, R10 to R7, R12 to R8, R13 to R9, U11 to U1, U12 to U2, U6 to U4, U7 to U5, U8 to U6, U9 to U7
Connections:
- net Net-(D2-A) renamed /MESA_P3_5V
- J4 pad 2_2: /MESA P3 REAR IO/IO_09_STEPGEN_02_STEP -> /MESA P3 REAR IO/IO_02_STEPGEN_00_STEP
- J4 pad 2_4: /MESA P3 REAR IO/IO_02_STEPGEN_00_STEP -> /MESA P3 REAR IO/IO_09_STEPGEN_02_STEP
- J4 pad 4_2: /MESA P3 REAR IO/IO_10_STEPGEN_02_DIR -> /MESA P3 REAR IO/IO_04_STEPGEN_00_DIR
- J4 pad 4_4: /MESA P3 REAR IO/IO_04_STEPGEN_00_DIR -> /MESA P3 REAR IO/IO_10_STEPGEN_02_DIR
- J4 pad 6_2: /Z MOT/ENABLE -> /X MOT/ENABLE
- J4 pad 6_4: /X MOT/ENABLE -> /Z MOT/ENABLE
- R19 pad 1: Net-(R23-Pad1) -> Net-(R19-Pad1)
- R3 pad 1: Net-(R4-Pad1) -> Net-(R3-Pad1)
- R5 pad 1: Net-(R7-Pad1) -> Net-(R5-Pad1)
- R7 pad 1: Net-(R10-Pad1) -> Net-(R7-Pad1)
- R9 pad 1: Net-(R13-Pad1) -> Net-(R9-Pad1)
- U1 pad 1: /LIM X/INPUT -> /DRAWBAR SW/INPUT
- U1 pad 2: Net-(R1-Pad1) -> Net-(R3-Pad1)
- U1 pad 3: Net-(R13-Pad1) -> Net-(R1-Pad1)
- U1 pad 4: /LIM Y/INPUT -> /LIM X/INPUT
- U1 pad 6: /LIMIT_Y -> /LIMIT_X
- U1 pad 7: /LIMIT_X -> /DRAWBAR_SW
- U2 pad 1: /LIM Z/INPUT -> /PROBE/INPUT
- U2 pad 2: Net-(R10-Pad1) -> Net-(R5-Pad1)
- U2 pad 3: Net-(R7-Pad1) -> Net-(R19-Pad1)
- U2 pad 4: /PROBE/INPUT -> /TOOL_PROBE/INPUT
- U2 pad 6: /PROBE -> /TOOL_PROBE
- U2 pad 7: /LIMIT_Z -> /PROBE
Routing:
- net +5VP: track 0.00 -> 257.9 mm
- net +24V: track 34.6 -> 202.5 mm
- net /DRAWBAR_VALVE: track 0.00 -> 131.7 mm, vias 0 -> 1
- net /MIST: track 0.00 -> 125.7 mm, vias 0 -> 1
- net /TOOL_PROBE: track 0.00 -> 104.9 mm, vias 0 -> 1
- net /ARGON ESTOP/ESTOP+: track 0.00 -> 104.0 mm
- net /MESA P3 REAR IO/IO_09_STEPGEN_02_STEP: track 0.00 -> 101.3 mm
- net /DRAWBAR_SW: track 0.00 -> 95.0 mm
- net /PENDANT_SELX: track 0.00 -> 92.1 mm
- net /MESA P3 REAR IO/IO_10_STEPGEN_02_DIR: track 0.00 -> 89.8 mm
- net /PENDANT_SELY: track 0.00 -> 84.4 mm
- net /LIMIT_X: track 0.00 -> 84.3 mm
- net /MESA P3 REAR IO/IO_06_STEPGEN_01_STEP: track 0.00 -> 81.2 mm
- net /PENDANT_SELZ: track 0.00 -> 80.3 mm
- net /MESA P3 REAR IO/IO_08_STEPGEN_01_DIR: track 0.00 -> 78.8 mm
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- added copper zone on B.Cu, net GND
Other:
- board size 149.9 x 127.1 mm -> 149.9 x 103 mm
- board text added: "ALL INPUTS OPTOISOLATED SINK"

Commit message: Couple of routes
Routing:
- net /ALARM: track 62.3 -> 222.0 mm, vias 3 -> 4
- net /AXIS_PWR: track 0.00 -> 112.9 mm, vias 0 -> 3
- net /MESA P2 INTERNAL IO/MESA_5V: track 56.4 -> 52.1 mm
- net Net-(R15-Pad2): track 0.00 -> 2.55 mm
- net Net-(R14-Pad2): track 0.00 -> 2.55 mm
- net Net-(R13-Pad2): track 0.00 -> 2.55 mm
- net /MIST: track 125.7 -> 128.1 mm

Commit message: Final tweaks for production
Parts:
- removed JP1: HSIN1, Connector_PinHeader_2.54mm:PinHeader_1x03_P2.54mm_Vertical
- removed JP2: HSIN2, Connector_PinHeader_2.54mm:PinHeader_1x03_P2.54mm_Vertical
Connections:
- J10 pad A14: /SPINDLE_PWM_SIG -> /MESA P3 REAR IO/IO_01_PWMGEN_00_PWM
- J10 pad A16: /SPINDLE_PWM_DIR -> /MESA P3 REAR IO/IO_05_PWMGEN_00_DIR
- J10 pad A8: /SPINDLE_STEPGEN_STEP -> /MESA P3 REAR IO/IO_11_STEPGEN_03_STEP
- J10 pad A9: /SPINDLE_STEPGEN_DIR -> /MESA P3 REAR IO/IO_12_STEPGEN_03_DIR
- J3 pad 4: Net-(J3-Pin_4) -> unconnected-(J3-Pin_4-Pad4)
- J3 pad 6: Net-(J3-Pin_6) -> unconnected-(J3-Pin_6-Pad6)
Routing:
- net /PROBE: track 48.3 -> 108.9 mm, vias 0 -> 2
- net /LIMIT_Y: track 39.8 -> 85.0 mm, vias 0 -> 2
- net Net-(J3-Pin_6): track 12.0 -> 0.00 mm
- net Net-(J3-Pin_4): track 8.14 -> 0.00 mm
- net /TOOL_PROBE: track 104.6 -> 109.1 mm
- net +24V: track 202.5 -> 205.3 mm
- net /SPINDLE_ENC_B: track 57.1 -> 55.6 mm
- net /MIST: track 128.1 -> 129.0 mm
- net /PENDANT_SELX: track 92.1 -> 92.8 mm
Other:
- board text removed: "PWM"
- board text removed: "SPINDLE SOURCE"
- board text removed: "STEPGEN"
