File: UnifiedBreakout/UnifiedBreakout/_autosave-UnifiedBreakout.sch (KiCad schematic (older format))
At the start: 37 parts, among them J1 24V DC IN, J2 ATX-24, J22 DRAWBAR, J23 MIST, J24 AXIS PWR IN, J25 AXIS PWR OUT, J3 5V BUS, J4 24V BUS, J5 12V BUS, U1 4N35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

Commit message: Finished(?) unified breakout layout
Parts:
- added H5, H6: MountingHole, MountingHole:MountingHole_3.2mm_M3, symbol Mechanical:MountingHole
Changed lines of the file:
@@
+	1    0    0    -1
+$EndComp
+$Comp
+L Mechanical:MountingHole H6
+U 1 1 5EAE25AF
+P 9150 10550
+F 0 "H6" H 9250 10596 50  0000 L CNN
+F 1 "MountingHole" H 9250 10505 50  0000 L CNN
+F 2 "MountingHole:MountingHole_3.2mm_M3" H 9150 10550 50  0001 C CNN
+F 3 "~" H 9150 10550 50  0001 C CNN
+	1    9150 10550
+	1    0    0    -1
+$EndComp
+$Comp
+L Mechanical:MountingHole H5
+U 1 1 5EAE2839
+P 8850 10750
+F 0 "H5" H 8950 10796 50  0000 L CNN
+F 1 "MountingHole" H 8950 10705 50  0000 L CNN
+F 2 "MountingHole:MountingHole_3.2mm_M3" H 8850 10750 50  0001 C CNN
+F 3 "~" H 8850 10750 50  0001 C CNN
+	1    8850 10750
 	1    0    0    -1
 $EndComp
