File: UnifiedBreakout/UnifiedBreakout/argon_encoder.sch (KiCad schematic (older format))
At the start: 3 parts, among them J12 ENCODER OUT, J13 ENCODER IN

Commit message: More placement, add some custom parts
Parts:
- J12: value ENCODER OUT -> ENCODER IN
- J13: value ENCODER IN -> ENCODER OUT
Changed lines of the file:
@@
 P 6100 3500
 F 0 "J13" H 6254 3502 50  0000 L CNN
-F 1 "ENCODER IN" H 6254 3411 50  0000 L CNN
+F 1 "ENCODER OUT" H 6254 3411 50  0000 L CNN
 F 2 "Connector_Dsub:DSUB-15_Female_Horizontal_P2.77x2.84mm_EdgePinOffset7.70mm_Housed_MountingHolesOffset9.12mm" H 6100 3500 50  0001 C CNN
 F 3 " ~" H 6100 3500 50  0001 C CNN
@@
 P 3800 3500
 F 0 "J12" H 3706 4492 50  0000 C CNN
-F 1 "ENCODER OUT" H 3706 4401 50  0000 C CNN
+F 1 "ENCODER IN" H 3706 4401 50  0000 C CNN
 F 2 "Connector_Dsub:DSUB-15_Female_Horizontal_P2.77x2.84mm_EdgePinOffset7.70mm_Housed_MountingHolesOffset9.12mm" H 3800 3500 50  0001 C CNN
 F 3 " ~" H 3800 3500 50  0001 C CNN

Commit message: Finished(?) unified breakout layout
Connections:
- net GND: now also J12.10 (P10)
Changed lines of the file:
@@
 Select between Argon 5V and Mesa 5V with this jumper
 Wire Wire Line
-	5300 4500 3800 4500
+	5300 4500 4350 4500
 Wire Wire Line
 	3800 4500 3800 4400
@@
 	4650 3600 4100 3600
 Connection ~ 4650 3600
+Wire Wire Line
+	4100 3100 4350 3100
+Wire Wire Line
+	4350 3100 4350 4500
+Connection ~ 4350 4500
+Wire Wire Line
+	4350 4500 3800 4500
 $EndSCHEMATC
