File: UnifiedBreakout/UnifiedBreakout/UnifiedBreakout.sch (KiCad schematic (older format))
At the start: 38 parts, among them J1 24V DC IN, J2 ATX-24, J22 DRAWBAR, J23 MIST, J24 AXIS PWR IN, J25 AXIS PWR OUT, J3 5V BUS, J4 24V BUS, J5 12V BUS, J6 ARGON RS485, U1 4N35, U7 74HC14

Commit message: Finished(?) unified breakout layout
Parts:
- removed J6: ARGON RS485, Connector_Phoenix_MSTB:PhoenixContact_MSTBA_2,5_3-G-5,08_1x03_P5.08mm_Horizontal, symbol Connector:Screw_Terminal_01x03
- added H? (x2): MountingHole, MountingHole:MountingHole_3.2mm_M3, symbol Mechanical:MountingHole
- added unit 7 of U7
Connections:
- net +5VP: now also U7.14 (VCC)
- net GND: now also U7.7 (GND)
Changed lines of the file:
@@
 LIMIT_Z
-$Comp
-L Connector:Screw_Terminal_01x03 J6
-U 1 1 5ED09EA9
-P 12500 9100
-F 0 "J6" H 12418 9417 50  0000 C CNN
-F 1 "ARGON RS485" H 12418 9326 50  0000 C CNN
-F 2 "Connector_Phoenix_MSTB:PhoenixContact_MSTBA_2,5_3-G-5,08_1x03_P5.08mm_Horizontal" H 12500 9100 50  0001 C CNN
-F 3 "~" H 12500 9100 50  0001 C CNN
-	1    12500 9100
-	-1   0    0    -1
-$EndComp
-Wire Wire Line
-	13650 9000 12700 9000
-Wire Wire Line
-	12700 9100 13650 9100
-$Comp
-L power:GND #PWR048
-U 1 1 5ED1E529
-P 12700 9200
-F 0 "#PWR048" H 12700 8950 50  0001 C CNN
-F 1 "GND" H 12705 9027 50  0000 C CNN
-F 2 "" H 12700 9200 50  0001 C CNN
-F 3 "" H 12700 9200 50  0001 C CNN
-	1    12700 9200
-	1    0    0    -1
-$EndComp
 $Comp
 L Connector:Screw_Terminal_01x02 J5
@@
 	7250 7350 7050 7350
 $Comp
+L power:GND #PWR0110
+U 1 1 5EBD0213
+P 7250 6050
+F 0 "#PWR0110" H 7250 5800 50  0001 C CNN
+F 1 "GND" H 7255 5877 50  0000 C CNN
+F 2 "" H 7250 6050 50  0001 C CNN
+F 3 "" H 7250 6050 50  0001 C CNN
+	1    7250 6050
+	1    0    0    -1
+$EndComp
+$Comp
+L power:+12V #PWR0111
+U 1 1 5EBD0601
+P 7500 5800
+F 0 "#PWR0111" H 7500 5650 50  0001 C CNN
+F 1 "+12V" H 7515 5973 50  0000 C CNN
+F 2 "" H 7500 5800 50  0001 C CNN
+F 3 "" H 7500 5800 50  0001 C CNN
+	1    7500 5800
+	1    0    0    -1
+$EndComp
+$Comp
+L power:+12V #PWR0112
+U 1 1 5EBD0AD9
+P 7500 7100
+F 0 "#PWR0112" H 7500 6950 50  0001 C CNN
+F 1 "+12V" H 7515 7273 50  0000 C CNN
+F 2 "" H 7500 7100 50  0001 C CNN
+F 3 "" H 7500 7100 50  0001 C CNN
+	1    7500 7100
+	1    0    0    -1
+$EndComp
+$Comp
+L Mechanical:MountingHole H1
+U 1 1 5E998E63
+P 8300 10200
+F 0 "H1" H 8400 10246 50  0000 L CNN
+F 1 "MountingHole" H 8400 10155 50  0000 L CNN
+F 2 "MountingHole:MountingHole_3.2mm_M3" H 8300 10200 50  0001 C CNN
+F 3 "~" H 8300 10200 50  0001 C CNN
+	1    8300 10200
+	1    0    0    -1
+$EndComp
+$Comp
+L Mechanical:MountingHole H2
+U 1 1 5E999355
+P 8650 10200
+F 0 "H2" H 8750 10246 50  0000 L CNN
+F 1 "MountingHole" H 8750 10155 50  0000 L CNN
+F 2 "MountingHole:MountingHole_3.2mm_M3" H 8650 10200 50  0001 C CNN
+F 3 "~" H 8650 10200 50  0001 C CNN
+	1    8650 10200
+	1    0    0    -1
+$EndComp
+$Comp
+L Mechanical:MountingHole H3
+U 1 1 5E9994FD
+P 8900 10200
+F 0 "H3" H 9000 10246 50  0000 L CNN
+F 1 "MountingHole" H 9000 10155 50  0000 L CNN
+F 2 "MountingHole:MountingHole_3.2mm_M3" H 8900 10200 50  0001 C CNN
+F 3 "~" H 8900 10200 50  0001 C CNN
+	1    8900 10200
+	1    0    0    -1
+$EndComp
+$Comp
+L Mechanical:MountingHole H4
+U 1 1 5E999660
+P 9150 10200
+F 0 "H4" H 9250 10246 50  0000 L CNN
+F 1 "MountingHole" H 9250 10155 50  0000 L CNN
+F 2 "MountingHole:MountingHole_3.2mm_M3" H 9150 10200 50  0001 C CNN
+F 3 "~" H 9150 10200 50  0001 C CNN
+	1    9150 10200
+	1    0    0    -1
+$EndComp
+$Comp
+L 74xx:74HC14 U7
+U 7 1 5EA1A05D
+P 5150 8700
+F 0 "U7" H 5150 9017 50  0000 C CNN
+F 1 "74HC14" H 5150 8926 50  0000 C CNN
+F 2 "Package_DIP:DIP-14_W7.62mm_LongPads" H 5150 8700 50  0001 C CNN
+F 3 "http://www.ti.com/lit/gpn/sn74HC14" H 5150 8700 50  0001 C CNN
+	7    5150 8700
+	1    0    0    -1
+$EndComp
+$Comp
+L power:+5VP #PWR0113
+U 1 1 5EA1AED5
+P 5150 8200
+F 0 "#PWR0113" H 5150 8050 50  0001 C CNN
+F 1 "+5VP" H 5165 8373 50  0000 C CNN
+F 2 "" H 5150 8200 50  0001 C CNN
+F 3 "" H 5150 8200 50  0001 C CNN
+	1    5150 8200
+	1    0    0    -1
+$EndComp
+$Comp
+L power:GND #PWR0114
+U 1 1 5EA1B659
+P 5150 9200
+F 0 "#PWR0114" H 5150 8950 50  0001 C CNN
+F 1 "GND" H 5155 9027 50  0000 C CNN
+F 2 "" H 5150 9200 50  0001 C CNN
+F 3 "" H 5150 9200 50  0001 C CNN
+	1    5150 9200
+	1    0    0    -1
+$EndComp
+$Comp
 L power:GND #PWR0109
 U 1 1 5EBCFE40
@@
 $EndComp
 $Comp
-L power:GND #PWR0110
-U 1 1 5EBD0213
-P 7250 6050
-F 0 "#PWR0110" H 7250 5800 50  0001 C CNN
-F 1 "GND" H 7255 5877 50  0000 C CNN
-F 2 "" H 7250 6050 50  0001 C CNN
-F 3 "" H 7250 6050 50  0001 C CNN
-	1    7250 6050
-	1    0    0    -1
-$EndComp
-$Comp
-L power:+12V #PWR0111
-U 1 1 5EBD0601
-P 7500 5800
-F 0 "#PWR0111" H 7500 5650 50  0001 C CNN
-F 1 "+12V" H 7515 5973 50  0000 C CNN
-F 2 "" H 7500 5800 50  0001 C CNN
-F 3 "" H 7500 5800 50  0001 C CNN
-	1    7500 5800
-	1    0    0    -1
-$EndComp
-$Comp
-L power:+12V #PWR0112
-U 1 1 5EBD0AD9
-P 7500 7100
-F 0 "#PWR0112" H 7500 6950 50  0001 C CNN
-F 1 "+12V" H 7515 7273 50  0000 C CNN
-F 2 "" H 7500 7100 50  0001 C CNN
-F 3 "" H 7500 7100 50  0001 C CNN
-	1    7500 7100
-	1    0    0    -1
-$EndComp
-$Comp
-L Mechanical:MountingHole H1
-U 1 1 5E998E63
-P 8300 10200
-F 0 "H1" H 8400 10246 50  0000 L CNN
-F 1 "MountingHole" H 8400 10155 50  0000 L CNN
-F 2 "MountingHole:MountingHole_3.2mm_M3" H 8300 10200 50  0001 C CNN
-F 3 "~" H 8300 10200 50  0001 C CNN
-	1    8300 10200
-	1    0    0    -1
-$EndComp
-$Comp
-L Mechanical:MountingHole H2
-U 1 1 5E999355
-P 8650 10200
-F 0 "H2" H 8750 10246 50  0000 L CNN
-F 1 "MountingHole" H 8750 10155 50  0000 L CNN
-F 2 "MountingHole:MountingHole_3.2mm_M3" H 8650 10200 50  0001 C CNN
-F 3 "~" H 8650 10200 50  0001 C CNN
-	1    8650 10200
-	1    0    0    -1
-$EndComp
-$Comp
-L Mechanical:MountingHole H3
-U 1 1 5E9994FD
-P 8900 10200
-F 0 "H3" H 9000 10246 50  0000 L CNN
-F 1 "MountingHole" H 9000 10155 50  0000 L CNN
-F 2 "MountingHole:MountingHole_3.2mm_M3" H 8900 10200 50  0001 C CNN
-F 3 "~" H 8900 10200 50  0001 C CNN
-	1    8900 10200
-	1    0    0    -1
-$EndComp
-$Comp
-L Mechanical:MountingHole H4
-U 1 1 5E999660
-P 9150 10200
-F 0 "H4" H 9250 10246 50  0000 L CNN
-F 1 "MountingHole" H 9250 10155 50  0000 L CNN
-F 2 "MountingHole:MountingHole_3.2mm_M3" H 9150 10200 50  0001 C CNN
-F 3 "~" H 9150 10200 50  0001 C CNN
-	1    9150 10200
-	1    0    0    -1
-$EndComp
+L Mechanical:MountingHole H?
+U 1 1 5EAE25AF
+P 9150 10550
+F 0 "H?" H 9250 10596 50  0000 L CNN
+F 1 "MountingHole" H 9250 10505 50  0000 L CNN
+F 2 "MountingHole:MountingHole_3.2mm_M3" H 9150 10550 50  0001 C CNN
+F 3 "~" H 9150 10550 50  0001 C CNN
+	1    9150 10550
+	1    0    0    -1
+$EndComp
+$Comp
+L Mechanical:MountingHole H?
+U 1 1 5EAE2839
+P 8850 10750
+F 0 "H?" H 8950 10796 50  0000 L CNN
+F 1 "MountingHole" H 8950 10705 50  0000 L CNN
+F 2 "MountingHole:MountingHole_3.2mm_M3" H 8850 10750 50  0001 C CNN
+F 3 "~" H 8850 10750 50  0001 C CNN
+	1    8850 10750
+	1    0    0    -1
+$EndComp

Commit message: Updated BOM
Parts:
- C2, C4, C6, C8: MPN 515D107M035BB6AE3 -> 860080574007; Manufacturer Vishay -> Wurth Elektronik
- J2: MPN (none) -> 39-30-1240; Manufacturer (none) -> Molex
- J22, J23, J3, J4, J5: MPN (none) -> 1757242; Manufacturer (none) -> Phoenix Contact
- J24, J25: MPN (none) -> 1757255; Manufacturer (none) -> Phoenix Contact
- gave numbers to parts that had none: 2
Changed lines of the file:
@@
 F 2 "Capacitor_THT:CP_Radial_D8.0mm_P3.50mm" H 4938 10500 50  0001 C CNN
 F 3 "~" H 4900 10650 50  0001 C CNN
-F 4 "515D107M035BB6AE3" H 4900 10650 50  0001 C CNN "MPN"
-F 5 "Vishay" H 4900 10650 50  0001 C CNN "Manufacturer"
+F 4 "860080574007" H 4900 10650 50  0001 C CNN "MPN"
+F 5 "Wurth Elektronik" H 4900 10650 50  0001 C CNN "Manufacturer"
 	1    4900 10650
 	1    0    0    -1
@@
 F 2 "Capacitor_THT:CP_Radial_D8.0mm_P3.50mm" H 3888 10500 50  0001 C CNN
 F 3 "~" H 3850 10650 50  0001 C CNN
-F 4 "515D107M035BB6AE3" H 3850 10650 50  0001 C CNN "MPN"
-F 5 "Vishay" H 3850 10650 50  0001 C CNN "Manufacturer"
+F 4 "860080574007" H 3850 10650 50  0001 C CNN "MPN"
+F 5 "Wurth Elektronik" H 3850 10650 50  0001 C CNN "Manufacturer"
 	1    3850 10650
 	1    0    0    -1
@@
 F 2 "Capacitor_THT:CP_Radial_D8.0mm_P3.50mm" H 5938 10500 50  0001 C CNN
 F 3 "~" H 5900 10650 50  0001 C CNN
-F 4 "515D107M035BB6AE3" H 5900 10650 50  0001 C CNN "MPN"
-F 5 "Vishay" H 5900 10650 50  0001 C CNN "Manufacturer"
+F 4 "860080574007" H 5900 10650 50  0001 C CNN "MPN"
+F 5 "Wurth Elektronik" H 5900 10650 50  0001 C CNN "Manufacturer"
 	1    5900 10650
 	1    0    0    -1
@@
 F 2 "Connector_Molex:Molex_Mini-Fit_Jr_5569-24A2_2x12_P4.20mm_Horizontal" H 2250 7750 50  0001 C CNN
 F 3 "https://www.intel.com/content/dam/www/public/us/en/documents/guides/power-supply-design-guide-june.pdf#page=33" H 4650 7300 50  0001 C CNN
+F 4 "39-30-1240" H 2250 7850 50  0001 C CNN "MPN"
+F 5 "Molex" H 2250 7850 50  0001 C CNN "Manufacturer"
 	1    2250 7850
 	1    0    0    -1
@@
 F 2 "Capacitor_THT:CP_Radial_D8.0mm_P3.50mm" H 6938 10500 50  0001 C CNN
 F 3 "~" H 6900 10650 50  0001 C CNN
-F 4 "515D107M035BB6AE3" H 6900 10650 50  0001 C CNN "MPN"
-F 5 "Vishay" H 6900 10650 50  0001 C CNN "Manufacturer"
+F 4 "860080574007" H 6900 10650 50  0001 C CNN "MPN"
+F 5 "Wurth Elektronik" H 6900 10650 50  0001 C CNN "Manufacturer"
 	1    6900 10650
 	1    0    0    -1
@@
 F 2 "Connector_Phoenix_MSTB:PhoenixContact_MSTBA_2,5_2-G-5,08_1x02_P5.08mm_Horizontal" H 2600 10600 50  0001 C CNN
 F 3 "~" H 2600 10600 50  0001 C CNN
+F 4 "1757242" H 2600 10600 50  0001 C CNN "MPN"
+F 5 "Phoenix Contact" H 2600 10600 50  0001 C CNN "Manufacturer"
 	1    2600 10600
 	1    0    0    -1
@@
 F 2 "Connector_Phoenix_MSTB:PhoenixContact_MSTBA_2,5_2-G-5,08_1x02_P5.08mm_Horizontal" H 1800 10600 50  0001 C CNN
 F 3 "~" H 1800 10600 50  0001 C CNN
+F 4 "1757242" H 1800 10600 50  0001 C CNN "MPN"
+F 5 "Phoenix Contact" H 1800 10600 50  0001 C CNN "Manufacturer"
 	1    1800 10600
 	1    0    0    -1
@@
 F 2 "Connector_Phoenix_MSTB:PhoenixContact_MSTBA_2,5_2-G-5,08_1x02_P5.08mm_Horizontal" H 1050 10600 50  0001 C CNN
 F 3 "~" H 1050 10600 50  0001 C CNN
+F 4 "1757242" H 1050 10600 50  0001 C CNN "MPN"
+F 5 "Phoenix Contact" H 1050 10600 50  0001 C CNN "Manufacturer"
 	1    1050 10600
 	1    0    0    -1
@@
 F 2 "Connector_Phoenix_MSTB:PhoenixContact_MSTBA_2,5_3-G-5,08_1x03_P5.08mm_Horizontal" H 8050 4600 50  0001 C CNN
 F 3 "~" H 8050 4600 50  0001 C CNN
+F 4 "1757255" H 8050 4600 50  0001 C CNN "MPN"
+F 5 "Phoenix Contact" H 8050 4600 50  0001 C CNN "Manufacturer"
 	1    8050 4600
 	1    0    0    -1
@@
 F 2 "Connector_Phoenix_MSTB:PhoenixContact_MSTBA_2,5_3-G-5,08_1x03_P5.08mm_Horizontal" H 8050 5150 50  0001 C CNN
 F 3 "~" H 8050 5150 50  0001 C CNN
+F 4 "1757255" H 8050 5150 50  0001 C CNN "MPN"
+F 5 "Phoenix Contact" H 8050 5150 50  0001 C CNN "Manufacturer"
 	1    8050 5150
 	1    0    0    -1
@@
 F 2 "Connector_Phoenix_MSTB:PhoenixContact_MSTBA_2,5_2-G-5,08_1x02_P5.08mm_Horizontal" H 7700 5800 50  0001 C CNN
 F 3 "~" H 7700 5800 50  0001 C CNN
+F 4 "1757242" H 7700 5800 50  0001 C CNN "MPN"
+F 5 "Phoenix Contact" H 7700 5800 50  0001 C CNN "Manufacturer"
 	1    7700 5800
 	1    0    0    -1
@@
 F 2 "Connector_Phoenix_MSTB:PhoenixContact_MSTBA_2,5_2-G-5,08_1x02_P5.08mm_Horizontal" H 7700 7100 50  0001 C CNN
 F 3 "~" H 7700 7100 50  0001 C CNN
+F 4 "1757242" H 7700 7100 50  0001 C CNN "MPN"
+F 5 "Phoenix Contact" H 7700 7100 50  0001 C CNN "Manufacturer"
 	1    7700 7100
 	1    0    0    -1
@@
 $EndComp
 $Comp
-L Mechanical:MountingHole H?
+L Mechanical:MountingHole H6
 U 1 1 5EAE25AF
 P 9150 10550
-F 0 "H?" H 9250 10596 50  0000 L CNN
+F 0 "H6" H 9250 10596 50  0000 L CNN
 F 1 "MountingHole" H 9250 10505 50  0000 L CNN
 F 2 "MountingHole:MountingHole_3.2mm_M3" H 9150 10550 50  0001 C CNN
@@
 $EndComp
 $Comp
-L Mechanical:MountingHole H?
+L Mechanical:MountingHole H5
 U 1 1 5EAE2839
 P 8850 10750
-F 0 "H?" H 8950 10796 50  0000 L CNN
+F 0 "H5" H 8950 10796 50  0000 L CNN
 F 1 "MountingHole" H 8950 10705 50  0000 L CNN
 F 2 "MountingHole:MountingHole_3.2mm_M3" H 8850 10750 50  0001 C CNN
