File: UnifiedBreakout/UnifiedBreakout/UnifiedBreakout.sch (KiCad schematic (older format))
At the start: 39 parts, among them J1 24V DC IN, J2 ATX-24, J22 DRAWBAR, J23 MIST, J24 AXIS PWR IN, J25 AXIS PWR OUT, J3 5V BUS, J4 24V BUS, J5 12V BUS, U1 4N35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

Commit message: Final updates to unified BoB
Parts:
- C1, C3, C5, C7: footprint Capacitor_THT:C_Disc_D5.0mm_W2.5mm_P2.50mm -> Capacitor_THT:C_Disc_D5.0mm_W2.5mm_P5.00mm
- R1, R2, R24, R25, R26, R3, R4, R5, R6, R7: footprint Resistor_THT:R_Axial_DIN0207_L6.3mm_D2.5mm_P10.16mm_Horizontal -> Resistor_THT:R_Axial_DIN0207_L6.3mm_D2.5mm_P7.62mm_Horizontal
Changed lines of the file:
@@
 F 0 "C3" H 4565 10696 50  0000 L CNN
 F 1 "100n" H 4565 10605 50  0000 L CNN
-F 2 "Capacitor_THT:C_Disc_D5.0mm_W2.5mm_P2.50mm" H 4488 10500 50  0001 C CNN
+F 2 "Capacitor_THT:C_Disc_D5.0mm_W2.5mm_P5.00mm" H 4488 10500 50  0001 C CNN
 F 3 "~" H 4450 10650 50  0001 C CNN
 F 4 "K104K15X7RF53H5" H 4450 10650 50  0001 C CNN "MPN"
@@
 F 0 "C1" H 3515 10696 50  0000 L CNN
 F 1 "100n" H 3515 10605 50  0000 L CNN
-F 2 "Capacitor_THT:C_Disc_D5.0mm_W2.5mm_P2.50mm" H 3438 10500 50  0001 C CNN
+F 2 "Capacitor_THT:C_Disc_D5.0mm_W2.5mm_P5.00mm" H 3438 10500 50  0001 C CNN
 F 3 "~" H 3400 10650 50  0001 C CNN
 F 4 "K104K15X7RF53H5" H 3400 10650 50  0001 C CNN "MPN"
@@
 F 0 "C5" H 5565 10696 50  0000 L CNN
 F 1 "100n" H 5565 10605 50  0000 L CNN
-F 2 "Capacitor_THT:C_Disc_D5.0mm_W2.5mm_P2.50mm" H 5488 10500 50  0001 C CNN
+F 2 "Capacitor_THT:C_Disc_D5.0mm_W2.5mm_P5.00mm" H 5488 10500 50  0001 C CNN
 F 3 "~" H 5450 10650 50  0001 C CNN
 F 4 "K104K15X7RF53H5" H 5450 10650 50  0001 C CNN "MPN"
@@
 F 0 "R4" V 3043 7450 50  0000 C CNN
 F 1 "220R" V 3134 7450 50  0000 C CNN
-F 2 "Resistor_THT:R_Axial_DIN0207_L6.3mm_D2.5mm_P10.16mm_Horizontal" V 3180 7450 50  0001 C CNN
+F 2 "Resistor_THT:R_Axial_DIN0207_L6.3mm_D2.5mm_P7.62mm_Horizontal" V 3180 7450 50  0001 C CNN
 F 3 "~" H 3250 7450 50  0001 C CNN
 F 4 "CFR-25JB-52-220R" H 3250 7450 50  0001 C CNN "MPN"
@@
 F 0 "R1" H 1620 7146 50  0000 L CNN
 F 1 "2K2" H 1620 7055 50  0000 L CNN
-F 2 "Resistor_THT:R_Axial_DIN0207_L6.3mm_D2.5mm_P10.16mm_Horizontal" V 1480 7100 50  0001 C CNN
+F 2 "Resistor_THT:R_Axial_DIN0207_L6.3mm_D2.5mm_P7.62mm_Horizontal" V 1480 7100 50  0001 C CNN
 F 3 "~" H 1550 7100 50  0001 C CNN
 F 4 "CFR-25JB-52-2K2" H 1550 7100 50  0001 C CNN "MPN"
@@
 F 0 "R5" V 3043 7850 50  0000 C CNN
 F 1 "220R" V 3134 7850 50  0000 C CNN
-F 2 "Resistor_THT:R_Axial_DIN0207_L6.3mm_D2.5mm_P10.16mm_Horizontal" V 3180 7850 50  0001 C CNN
+F 2 "Resistor_THT:R_Axial_DIN0207_L6.3mm_D2.5mm_P7.62mm_Horizontal" V 3180 7850 50  0001 C CNN
 F 3 "~" H 3250 7850 50  0001 C CNN
 F 4 "CFR-25JB-52-220R" H 3250 7850 50  0001 C CNN "MPN"
@@
 F 0 "C7" H 6565 10696 50  0000 L CNN
 F 1 "100n" H 6565 10605 50  0000 L CNN
-F 2 "Capacitor_THT:C_Disc_D5.0mm_W2.5mm_P2.50mm" H 6488 10500 50  0001 C CNN
+F 2 "Capacitor_THT:C_Disc_D5.0mm_W2.5mm_P5.00mm" H 6488 10500 50  0001 C CNN
 F 3 "~" H 6450 10650 50  0001 C CNN
 F 4 "K104K15X7RF53H5" H 6450 10650 50  0001 C CNN "MPN"
@@
 F 0 "R2" V 1257 2500 50  0000 C CNN
 F 1 "220R" V 1166 2500 50  0000 C CNN
-F 2 "Resistor_THT:R_Axial_DIN0207_L6.3mm_D2.5mm_P10.16mm_Horizontal" V 980 2500 50  0001 C CNN
+F 2 "Resistor_THT:R_Axial_DIN0207_L6.3mm_D2.5mm_P7.62mm_Horizontal" V 980 2500 50  0001 C CNN
 F 3 "~" H 1050 2500 50  0001 C CNN
 F 4 "CFR-25JB-52-220R" H 1050 2500 50  0001 C CNN "MPN"
@@
 F 0 "R3" V 993 5300 50  0000 C CNN
 F 1 "220R" V 1084 5300 50  0000 C CNN
-F 2 "Resistor_THT:R_Axial_DIN0207_L6.3mm_D2.5mm_P10.16mm_Horizontal" V 1130 5300 50  0001 C CNN
+F 2 "Resistor_THT:R_Axial_DIN0207_L6.3mm_D2.5mm_P7.62mm_Horizontal" V 1130 5300 50  0001 C CNN
 F 3 "~" H 1200 5300 50  0001 C CNN
 F 4 "CFR-25JB-52-220R" H 1200 5300 50  0001 C CNN "MPN"
@@
 F 0 "R6" H 11820 8396 50  0000 L CNN
 F 1 "220K" H 11820 8305 50  0000 L CNN
-F 2 "Resistor_THT:R_Axial_DIN0207_L6.3mm_D2.5mm_P10.16mm_Horizontal" V 11680 8350 50  0001 C CNN
+F 2 "Resistor_THT:R_Axial_DIN0207_L6.3mm_D2.5mm_P7.62mm_Horizontal" V 11680 8350 50  0001 C CNN
 F 3 "~" H 11750 8350 50  0001 C CNN
 F 4 "CFR-25JB-52-220K" H 11750 8350 50  0001 C CNN "MPN"
@@
 F 0 "R7" V 12693 8100 50  0000 C CNN
 F 1 "2K2" V 12784 8100 50  0000 C CNN
-F 2 "Resistor_THT:R_Axial_DIN0207_L6.3mm_D2.5mm_P10.16mm_Horizontal" V 12830 8100 50  0001 C CNN
+F 2 "Resistor_THT:R_Axial_DIN0207_L6.3mm_D2.5mm_P7.62mm_Horizontal" V 12830 8100 50  0001 C CNN
 F 3 "~" H 12900 8100 50  0001 C CNN
 F 4 "CFR-25JB-52-2K2" H 12900 8100 50  0001 C CNN "MPN"
@@
 F 0 "R24" H 5270 4646 50  0000 L CNN
 F 1 "10K" H 5270 4555 50  0000 L CNN
-F 2 "Resistor_THT:R_Axial_DIN0207_L6.3mm_D2.5mm_P10.16mm_Horizontal" V 5130 4600 50  0001 C CNN
+F 2 "Resistor_THT:R_Axial_DIN0207_L6.3mm_D2.5mm_P7.62mm_Horizontal" V 5130 4600 50  0001 C CNN
 F 3 "~" H 5200 4600 50  0001 C CNN
 F 4 "CFR-25JB-52-10K " H 5200 4600 50  0001 C CNN "MPN"
@@
 F 0 "R25" H 5270 5946 50  0000 L CNN
 F 1 "10K" H 5270 5855 50  0000 L CNN
-F 2 "Resistor_THT:R_Axial_DIN0207_L6.3mm_D2.5mm_P10.16mm_Horizontal" V 5130 5900 50  0001 C CNN
+F 2 "Resistor_THT:R_Axial_DIN0207_L6.3mm_D2.5mm_P7.62mm_Horizontal" V 5130 5900 50  0001 C CNN
 F 3 "~" H 5200 5900 50  0001 C CNN
 F 4 "CFR-25JB-52-10K " H 5200 5900 50  0001 C CNN "MPN"
@@
 F 0 "R26" H 5270 7246 50  0000 L CNN
 F 1 "10K" H 5270 7155 50  0000 L CNN
-F 2 "Resistor_THT:R_Axial_DIN0207_L6.3mm_D2.5mm_P10.16mm_Horizontal" V 5130 7200 50  0001 C CNN
+F 2 "Resistor_THT:R_Axial_DIN0207_L6.3mm_D2.5mm_P7.62mm_Horizontal" V 5130 7200 50  0001 C CNN
 F 3 "~" H 5200 7200 50  0001 C CNN
 F 4 "CFR-25JB-52-10K " H 5200 7200 50  0001 C CNN "MPN"
