File: UnifiedBreakout/UnifiedBreakout/jog_pendant.sch (KiCad schematic (older format))
At the start: 1 part, among them J21 PENDANT

Commit message: Updated BOM
Parts:
- J21: Alternative MPN (none) -> L77SDB25SA4CH4F; MPN (none) -> ID25S33E4GX00LF; Manufacturer (none) -> Amphenol
Changed lines of the file:
@@
 F 2 "Connector_Dsub:DSUB-25_Female_Horizontal_P2.77x2.84mm_EdgePinOffset7.70mm_Housed_MountingHolesOffset9.12mm" H 5650 3650 50  0001 C CNN
 F 3 " ~" H 5650 3650 50  0001 C CNN
+F 4 "L77SDB25SA4CH4F " H 5650 3650 50  0001 C CNN "Alternative MPN"
+F 5 "ID25S33E4GX00LF" H 5650 3650 50  0001 C CNN "MPN"
+F 6 "Amphenol" H 5650 3650 50  0001 C CNN "Manufacturer"
 	1    5650 3650
 	1    0    0    -1
