File: UnifiedBreakout/UnifiedBreakout/argon_io.sch (KiCad schematic (older format))
At the start: 3 parts, among them J14 ARGON J5

Commit message: Invert outputs for active low, other cleanup
Parts:
- J14: footprint Connector_IDC:IDC-Header_2x13_P2.54mm_Vertical -> Connector_IDC:IDC-Header_2x13_P2.54mm_Horizontal
Connections:
- net GND: now also J14.15 (Pin_15)
- net GPI1: no longer names the net of J14.20 (Pin_20)
- net GPI2: no longer names the net of J14.22 (Pin_22)
- net GPI3: no longer names the net of J14.24 (Pin_24)
- net GPI4: no longer names the net of J14.26 (Pin_26)
- net GPO1: no longer names the net of J14.12 (Pin_12)
- net GPO2: no longer names the net of J14.14 (Pin_14)
- net GPO3 renamed FAULT
- net GPO4: no longer names the net of J14.18 (Pin_18)
Changed lines of the file:
@@
 $Descr A4 11693 8268
 encoding utf-8
-Sheet 11 20
+Sheet 11 18
 Title ""
 Date ""
@@
 F 0 "J14" H 5300 4417 50  0000 C CNN
 F 1 "ARGON J5" H 5300 4326 50  0000 C CNN
-F 2 "Connector_IDC:IDC-Header_2x13_P2.54mm_Vertical" H 5250 3600 50  0001 C CNN
+F 2 "Connector_IDC:IDC-Header_2x13_P2.54mm_Horizontal" H 5250 3600 50  0001 C CNN
 F 3 "~" H 5250 3600 50  0001 C CNN
 	1    5250 3600
 	1    0    0    -1
 $EndComp
-Text HLabel 5050 3000 0    50   Output ~ 0
+Text HLabel 4600 3000 0    50   Output ~ 0
 GND
-Text HLabel 5550 3500 2    50   Input ~ 0
-GPO1
-Text HLabel 5550 3600 2    50   Input ~ 0
-GPO2
-Text HLabel 5550 3700 2    50   Input ~ 0
-GPO3
-Text HLabel 5550 3800 2    50   Input ~ 0
-GPO4
-Text HLabel 5550 3900 2    50   Input ~ 0
-GPI1
-Text HLabel 5550 4000 2    50   Input ~ 0
-GPI2
-Text HLabel 5550 4100 2    50   Input ~ 0
-GPI3
-Text HLabel 5550 4200 2    50   Input ~ 0
-GPI4
 Text HLabel 7250 2850 2    50   Input ~ 0
 STEPGEN_STEP
@@
 Wire Wire Line
 	5550 3200 7000 3200
+Wire Wire Line
+	5050 3000 4800 3000
+Wire Wire Line
+	5050 3700 4800 3700
+Wire Wire Line
+	4800 3700 4800 3000
+Connection ~ 4800 3000
+Wire Wire Line
+	4800 3000 4600 3000
+Text HLabel 5550 3700 2    50   Input ~ 0
+FAULT
 $EndSCHEMATC

Commit message: Updated BOM
Parts:
- J14: MPN (none) -> 90130-3126; Manufacturer (none) -> Molex
Changed lines of the file:
@@
 F 2 "Connector_IDC:IDC-Header_2x13_P2.54mm_Horizontal" H 5250 3600 50  0001 C CNN
 F 3 "~" H 5250 3600 50  0001 C CNN
+F 4 "90130-3126 " H 5250 3600 50  0001 C CNN "MPN"
+F 5 "Molex" H 5250 3600 50  0001 C CNN "Manufacturer"
 	1    5250 3600
 	1    0    0    -1

Commit message: Final updates to unified BoB
Parts:
- J14: MPN 90130-3126 -> N2526-5002RB; Manufacturer Molex -> 3M
Changed lines of the file:
@@
 F 2 "Connector_IDC:IDC-Header_2x13_P2.54mm_Horizontal" H 5250 3600 50  0001 C CNN
 F 3 "~" H 5250 3600 50  0001 C CNN
-F 4 "90130-3126 " H 5250 3600 50  0001 C CNN "MPN"
-F 5 "Molex" H 5250 3600 50  0001 C CNN "Manufacturer"
+F 4 "N2526-5002RB" H 5250 3600 50  0001 C CNN "MPN"
+F 5 "3M" H 5250 3600 50  0001 C CNN "Manufacturer"
 	1    5250 3600
 	1    0    0    -1
