File: UnifiedBreakout/UnifiedBreakout/opto_input.sch (KiCad schematic (older format))
At the start: 4 parts, among them J16 RJ14, U2 4N35

Commit message: Invert outputs for active low, other cleanup
Changed lines of the file:
@@
 $Descr A4 11693 8268
 encoding utf-8
-Sheet 20 20
+Sheet 17 18
 Title ""
 Date ""
@@
 AR Path="/5E9DEC5E/5EA62D6B" Ref="U7"  Part="1"
 AR Path="/5E9DEC7B/5EA62D6B" Ref="U8"  Part="1"
-F 0 "U8" H 5750 3825 50  0000 C CNN
+F 0 "U6" H 5750 3825 50  0000 C CNN
 F 1 "4N35" H 5750 3734 50  0000 C CNN
 F 2 "Package_DIP:DIP-6_W7.62mm" H 5550 3300 50  0001 L CIN
@@
 AR Path="/5E9DEC5E/5EA63E66" Ref="R24"  Part="1"
 AR Path="/5E9DEC7B/5EA63E66" Ref="R26"  Part="1"
-F 0 "R26" H 5320 3946 50  0000 L CNN
+F 0 "R22" H 5320 3946 50  0000 L CNN
 F 1 "2K2" H 5320 3855 50  0000 L CNN
 F 2 "Resistor_THT:R_Axial_DIN0207_L6.3mm_D2.5mm_P10.16mm_Horizontal" V 5180 3900 50  0001 C CNN
@@
 AR Path="/5E9DEC5E/5EA649A8" Ref="J22"  Part="1"
 AR Path="/5E9DEC7B/5EA649A8" Ref="J23"  Part="1"
-F 0 "J23" H 3421 3304 50  0000 R CNN
+F 0 "J20" H 3421 3304 50  0000 R CNN
 F 1 "RJ14" H 3421 3395 50  0000 R CNN
 F 2 "Connector_RJ:RJ12_Amphenol_54601" V 3750 3325 50  0001 C CNN
@@
 AR Path="/5E9DEC5E/5EA66D61" Ref="R25"  Part="1"
 AR Path="/5E9DEC7B/5EA66D61" Ref="R27"  Part="1"
-F 0 "R27" H 6220 3946 50  0000 L CNN
+F 0 "R23" H 6220 3946 50  0000 L CNN
 F 1 "220K" H 6220 3855 50  0000 L CNN
 F 2 "Resistor_THT:R_Axial_DIN0207_L6.3mm_D2.5mm_P10.16mm_Horizontal" V 6080 3900 50  0001 C CNN

Commit message: Add extra pullups on inputs
Parts:
- added R27: 10K, Resistor_THT:R_Axial_DIN0207_L6.3mm_D2.5mm_P10.16mm_Horizontal, symbol Device:R
Connections:
- net SIGNAL: now also R27.2
- new net MESA_5V: R27.1
Changed lines of the file:
@@
 $Descr A4 11693 8268
 encoding utf-8
-Sheet 17 18
+Sheet 13 18
 Title ""
 Date ""
@@
 AR Path="/5E9DEC5E/5EA62D6B" Ref="U7"  Part="1"
 AR Path="/5E9DEC7B/5EA62D6B" Ref="U8"  Part="1"
-F 0 "U6" H 5750 3825 50  0000 C CNN
+F 0 "U2" H 5750 3825 50  0000 C CNN
 F 1 "4N35" H 5750 3734 50  0000 C CNN
 F 2 "Package_DIP:DIP-6_W7.62mm" H 5550 3300 50  0001 L CIN
@@
 AR Path="/5E9DEC5E/5EA63E66" Ref="R24"  Part="1"
 AR Path="/5E9DEC7B/5EA63E66" Ref="R26"  Part="1"
-F 0 "R22" H 5320 3946 50  0000 L CNN
+F 0 "R14" H 5320 3946 50  0000 L CNN
 F 1 "2K2" H 5320 3855 50  0000 L CNN
 F 2 "Resistor_THT:R_Axial_DIN0207_L6.3mm_D2.5mm_P10.16mm_Horizontal" V 5180 3900 50  0001 C CNN
@@
 AR Path="/5E9DEC5E/5EA649A8" Ref="J22"  Part="1"
 AR Path="/5E9DEC7B/5EA649A8" Ref="J23"  Part="1"
-F 0 "J20" H 3421 3304 50  0000 R CNN
+F 0 "J16" H 3421 3304 50  0000 R CNN
 F 1 "RJ14" H 3421 3395 50  0000 R CNN
 F 2 "Connector_RJ:RJ12_Amphenol_54601" V 3750 3325 50  0001 C CNN
@@
 AR Path="/5E9DEC5E/5EA66D61" Ref="R25"  Part="1"
 AR Path="/5E9DEC7B/5EA66D61" Ref="R27"  Part="1"
-F 0 "R23" H 6220 3946 50  0000 L CNN
+F 0 "R15" H 6220 3946 50  0000 L CNN
 F 1 "220K" H 6220 3855 50  0000 L CNN
 F 2 "Resistor_THT:R_Axial_DIN0207_L6.3mm_D2.5mm_P10.16mm_Horizontal" V 6080 3900 50  0001 C CNN
@@
 SIGNAL
 Wire Wire Line
-	6050 3500 6400 3500
+	6050 3500 6300 3500
 Wire Wire Line
 	6150 4050 6150 4300
@@
 Text HLabel 4150 3500 2    50   UnSpc ~ 0
 GND
+$Comp
+L Device:R R27
+U 1 1 5E9E2B63
+P 6300 3050
+AR Path="/5EA623AE/5E9E2B63" Ref="R27"  Part="1"
+AR Path="/5EA7F263/5E9E2B63" Ref="R28"  Part="1"
+AR Path="/5EA816C6/5E9E2B63" Ref="R29"  Part="1"
+AR Path="/5EA83CCC/5E9E2B63" Ref="R30"  Part="1"
+AR Path="/5EA86618/5E9E2B63" Ref="R31"  Part="1"
+F 0 "R27" H 6370 3096 50  0000 L CNN
+F 1 "10K" H 6370 3005 50  0000 L CNN
+F 2 "Resistor_THT:R_Axial_DIN0207_L6.3mm_D2.5mm_P10.16mm_Horizontal" V 6230 3050 50  0001 C CNN
+F 3 "~" H 6300 3050 50  0001 C CNN
+	1    6300 3050
+	1    0    0    -1
+$EndComp
+Wire Wire Line
+	6300 3200 6300 3500
+Connection ~ 6300 3500
+Wire Wire Line
+	6300 3500 6400 3500
+Text HLabel 6300 2900 1    50   UnSpc ~ 0
+MESA_5V
 $EndSCHEMATC

Commit message: Connectors placed
Parts:
- J16: footprint Connector_RJ:RJ12_Amphenol_54601 -> Connector_RJ:RJ14_Connfly_DS1133-S4_Horizontal
Changed lines of the file:
@@
 $Descr A4 11693 8268
 encoding utf-8
-Sheet 13 18
+Sheet 14 18
 Title ""
 Date ""
@@
 AR Path="/5E9DEC5E/5EA62D6B" Ref="U7"  Part="1"
 AR Path="/5E9DEC7B/5EA62D6B" Ref="U8"  Part="1"
-F 0 "U2" H 5750 3825 50  0000 C CNN
+F 0 "U6" H 5750 3825 50  0000 C CNN
 F 1 "4N35" H 5750 3734 50  0000 C CNN
 F 2 "Package_DIP:DIP-6_W7.62mm" H 5550 3300 50  0001 L CIN
@@
 AR Path="/5E9DEC5E/5EA63E66" Ref="R24"  Part="1"
 AR Path="/5E9DEC7B/5EA63E66" Ref="R26"  Part="1"
-F 0 "R14" H 5320 3946 50  0000 L CNN
+F 0 "R22" H 5320 3946 50  0000 L CNN
 F 1 "2K2" H 5320 3855 50  0000 L CNN
 F 2 "Resistor_THT:R_Axial_DIN0207_L6.3mm_D2.5mm_P10.16mm_Horizontal" V 5180 3900 50  0001 C CNN
@@
 AR Path="/5E9DEC5E/5EA649A8" Ref="J22"  Part="1"
 AR Path="/5E9DEC7B/5EA649A8" Ref="J23"  Part="1"
-F 0 "J16" H 3421 3304 50  0000 R CNN
+F 0 "J20" H 3421 3304 50  0000 R CNN
 F 1 "RJ14" H 3421 3395 50  0000 R CNN
-F 2 "Connector_RJ:RJ12_Amphenol_54601" V 3750 3325 50  0001 C CNN
+F 2 "Connector_RJ:RJ14_Connfly_DS1133-S4_Horizontal" V 3750 3325 50  0001 C CNN
 F 3 "~" V 3750 3325 50  0001 C CNN
 	1    3750 3300
@@
 AR Path="/5E9DEC5E/5EA66D61" Ref="R25"  Part="1"
 AR Path="/5E9DEC7B/5EA66D61" Ref="R27"  Part="1"
-F 0 "R15" H 6220 3946 50  0000 L CNN
+F 0 "R23" H 6220 3946 50  0000 L CNN
 F 1 "220K" H 6220 3855 50  0000 L CNN
 F 2 "Resistor_THT:R_Axial_DIN0207_L6.3mm_D2.5mm_P10.16mm_Horizontal" V 6080 3900 50  0001 C CNN
@@
 AR Path="/5EA83CCC/5E9E2B63" Ref="R30"  Part="1"
 AR Path="/5EA86618/5E9E2B63" Ref="R31"  Part="1"
-F 0 "R27" H 6370 3096 50  0000 L CNN
+F 0 "R31" H 6370 3096 50  0000 L CNN
 F 1 "10K" H 6370 3005 50  0000 L CNN
 F 2 "Resistor_THT:R_Axial_DIN0207_L6.3mm_D2.5mm_P10.16mm_Horizontal" V 6230 3050 50  0001 C CNN

Commit message: More placement, add some custom parts
Parts:
- J16: footprint Connector_RJ:RJ14_Connfly_DS1133-S4_Horizontal -> Wurth:615004141121
Changed lines of the file:
@@
 AR Path="/5E9DEC5E/5EA62D6B" Ref="U7"  Part="1"
 AR Path="/5E9DEC7B/5EA62D6B" Ref="U8"  Part="1"
-F 0 "U6" H 5750 3825 50  0000 C CNN
+F 0 "U3" H 5750 3825 50  0000 C CNN
 F 1 "4N35" H 5750 3734 50  0000 C CNN
 F 2 "Package_DIP:DIP-6_W7.62mm" H 5550 3300 50  0001 L CIN
@@
 AR Path="/5E9DEC5E/5EA63E66" Ref="R24"  Part="1"
 AR Path="/5E9DEC7B/5EA63E66" Ref="R26"  Part="1"
-F 0 "R22" H 5320 3946 50  0000 L CNN
+F 0 "R16" H 5320 3946 50  0000 L CNN
 F 1 "2K2" H 5320 3855 50  0000 L CNN
 F 2 "Resistor_THT:R_Axial_DIN0207_L6.3mm_D2.5mm_P10.16mm_Horizontal" V 5180 3900 50  0001 C CNN
@@
 AR Path="/5E9DEC5E/5EA649A8" Ref="J22"  Part="1"
 AR Path="/5E9DEC7B/5EA649A8" Ref="J23"  Part="1"
-F 0 "J20" H 3421 3304 50  0000 R CNN
+F 0 "J17" H 3421 3304 50  0000 R CNN
 F 1 "RJ14" H 3421 3395 50  0000 R CNN
-F 2 "Connector_RJ:RJ14_Connfly_DS1133-S4_Horizontal" V 3750 3325 50  0001 C CNN
+F 2 "Wurth:615004141121" V 3750 3325 50  0001 C CNN
 F 3 "~" V 3750 3325 50  0001 C CNN
 	1    3750 3300
@@
 AR Path="/5E9DEC5E/5EA66D61" Ref="R25"  Part="1"
 AR Path="/5E9DEC7B/5EA66D61" Ref="R27"  Part="1"
-F 0 "R23" H 6220 3946 50  0000 L CNN
+F 0 "R17" H 6220 3946 50  0000 L CNN
 F 1 "220K" H 6220 3855 50  0000 L CNN
 F 2 "Resistor_THT:R_Axial_DIN0207_L6.3mm_D2.5mm_P10.16mm_Horizontal" V 6080 3900 50  0001 C CNN
@@
 AR Path="/5EA83CCC/5E9E2B63" Ref="R30"  Part="1"
 AR Path="/5EA86618/5E9E2B63" Ref="R31"  Part="1"
-F 0 "R31" H 6370 3096 50  0000 L CNN
+F 0 "R28" H 6370 3096 50  0000 L CNN
 F 1 "10K" H 6370 3005 50  0000 L CNN
 F 2 "Resistor_THT:R_Axial_DIN0207_L6.3mm_D2.5mm_P10.16mm_Horizontal" V 6230 3050 50  0001 C CNN

Commit message: Assigned some parts
Parts:
- J16: MPN (none) -> 615004141121; Manufacturer (none) -> Wurth
- R14: MPN (none) -> CFR-25JB-52-2K2; Manufacturer (none) -> Yageo
- R15: MPN (none) -> CFR-25JB-52-220K; Manufacturer (none) -> Yageo
- R27: MPN (none) -> CFR-25JB-52-10K; Manufacturer (none) -> Yageo
- U2: MPN (none) -> 4N35; Manufacturer (none) -> Vishay
Changed lines of the file:
@@
 F 2 "Package_DIP:DIP-6_W7.62mm" H 5550 3300 50  0001 L CIN
 F 3 "https://www.vishay.com/docs/81181/4n35.pdf" H 5750 3500 50  0001 L CNN
+F 4 "4N35" H 5750 3500 50  0001 C CNN "MPN"
+F 5 "Vishay" H 5750 3500 50  0001 C CNN "Manufacturer"
 	1    5750 3500
 	1    0    0    -1
@@
 F 2 "Resistor_THT:R_Axial_DIN0207_L6.3mm_D2.5mm_P10.16mm_Horizontal" V 5180 3900 50  0001 C CNN
 F 3 "~" H 5250 3900 50  0001 C CNN
+F 4 "CFR-25JB-52-2K2" H 5250 3900 50  0001 C CNN "MPN"
+F 5 "Yageo" H 5250 3900 50  0001 C CNN "Manufacturer"
 	1    5250 3900
 	1    0    0    -1
@@
 F 2 "Wurth:615004141121" V 3750 3325 50  0001 C CNN
 F 3 "~" V 3750 3325 50  0001 C CNN
+F 4 "615004141121" H 3750 3300 50  0001 C CNN "MPN"
+F 5 "Wurth" H 3750 3300 50  0001 C CNN "Manufacturer"
 	1    3750 3300
 	1    0    0    1
@@
 F 2 "Resistor_THT:R_Axial_DIN0207_L6.3mm_D2.5mm_P10.16mm_Horizontal" V 6080 3900 50  0001 C CNN
 F 3 "~" H 6150 3900 50  0001 C CNN
+F 4 "CFR-25JB-52-220K" H 6150 3900 50  0001 C CNN "MPN"
+F 5 "Yageo" H 6150 3900 50  0001 C CNN "Manufacturer"
 	1    6150 3900
 	1    0    0    -1
@@
 F 2 "Resistor_THT:R_Axial_DIN0207_L6.3mm_D2.5mm_P10.16mm_Horizontal" V 6230 3050 50  0001 C CNN
 F 3 "~" H 6300 3050 50  0001 C CNN
+F 4 "CFR-25JB-52-10K " H 6300 3050 50  0001 C CNN "MPN"
+F 5 "Yageo" H 6300 3050 50  0001 C CNN "Manufacturer"
 	1    6300 3050
 	1    0    0    -1

Commit message: Finished(?) unified breakout layout
Connections:
- net GND: now also J16.3; no longer J16.4
- net at U2.1: now also J16.4; no longer J16.3
Changed lines of the file:
@@
 $Descr A4 11693 8268
 encoding utf-8
-Sheet 14 18
+Sheet 13 18
 Title ""
 Date ""
@@
 AR Path="/5E9DEC5E/5EA62D6B" Ref="U7"  Part="1"
 AR Path="/5E9DEC7B/5EA62D6B" Ref="U8"  Part="1"
-F 0 "U3" H 5750 3825 50  0000 C CNN
+F 0 "U2" H 5750 3825 50  0000 C CNN
 F 1 "4N35" H 5750 3734 50  0000 C CNN
 F 2 "Package_DIP:DIP-6_W7.62mm" H 5550 3300 50  0001 L CIN
@@
 AR Path="/5E9DEC5E/5EA63E66" Ref="R24"  Part="1"
 AR Path="/5E9DEC7B/5EA63E66" Ref="R26"  Part="1"
-F 0 "R16" H 5320 3946 50  0000 L CNN
+F 0 "R14" H 5320 3946 50  0000 L CNN
 F 1 "2K2" H 5320 3855 50  0000 L CNN
 F 2 "Resistor_THT:R_Axial_DIN0207_L6.3mm_D2.5mm_P10.16mm_Horizontal" V 5180 3900 50  0001 C CNN
@@
 AR Path="/5E9DEC5E/5EA649A8" Ref="J22"  Part="1"
 AR Path="/5E9DEC7B/5EA649A8" Ref="J23"  Part="1"
-F 0 "J17" H 3421 3304 50  0000 R CNN
+F 0 "J16" H 3421 3304 50  0000 R CNN
 F 1 "RJ14" H 3421 3395 50  0000 R CNN
 F 2 "Wurth:615004141121" V 3750 3325 50  0001 C CNN
@@
 AR Path="/5E9DEC5E/5EA66D61" Ref="R25"  Part="1"
 AR Path="/5E9DEC7B/5EA66D61" Ref="R27"  Part="1"
-F 0 "R17" H 6220 3946 50  0000 L CNN
+F 0 "R15" H 6220 3946 50  0000 L CNN
 F 1 "220K" H 6220 3855 50  0000 L CNN
 F 2 "Resistor_THT:R_Axial_DIN0207_L6.3mm_D2.5mm_P10.16mm_Horizontal" V 6080 3900 50  0001 C CNN
@@
 Wire Wire Line
 	5250 4300 5250 4050
-Wire Wire Line
-	4150 3400 5450 3400
 Text HLabel 4150 3300 2    50   UnSpc ~ 0
 24V
 Text HLabel 4150 3200 2    50   UnSpc ~ 0
 5V
-Text HLabel 4150 3500 2    50   UnSpc ~ 0
+Text HLabel 4150 3400 2    50   UnSpc ~ 0
 GND
 $Comp
@@
 AR Path="/5EA83CCC/5E9E2B63" Ref="R30"  Part="1"
 AR Path="/5EA86618/5E9E2B63" Ref="R31"  Part="1"
-F 0 "R28" H 6370 3096 50  0000 L CNN
+F 0 "R27" H 6370 3096 50  0000 L CNN
 F 1 "10K" H 6370 3005 50  0000 L CNN
 F 2 "Resistor_THT:R_Axial_DIN0207_L6.3mm_D2.5mm_P10.16mm_Horizontal" V 6230 3050 50  0001 C CNN
@@
 Text HLabel 6300 2900 1    50   UnSpc ~ 0
 MESA_5V
+Wire Wire Line
+	4150 3500 5050 3500
+Wire Wire Line
+	5050 3500 5050 3400
+Wire Wire Line
+	5050 3400 5450 3400
 $EndSCHEMATC

Commit message: Updated BOM
Changed lines of the file:
@@
 AR Path="/5E9DEC5E/5EA62D6B" Ref="U7"  Part="1"
 AR Path="/5E9DEC7B/5EA62D6B" Ref="U8"  Part="1"
-F 0 "U2" H 5750 3825 50  0000 C CNN
+F 0 "U6" H 5750 3825 50  0000 C CNN
 F 1 "4N35" H 5750 3734 50  0000 C CNN
 F 2 "Package_DIP:DIP-6_W7.62mm" H 5550 3300 50  0001 L CIN
@@
 AR Path="/5E9DEC5E/5EA63E66" Ref="R24"  Part="1"
 AR Path="/5E9DEC7B/5EA63E66" Ref="R26"  Part="1"
-F 0 "R14" H 5320 3946 50  0000 L CNN
+F 0 "R22" H 5320 3946 50  0000 L CNN
 F 1 "2K2" H 5320 3855 50  0000 L CNN
 F 2 "Resistor_THT:R_Axial_DIN0207_L6.3mm_D2.5mm_P10.16mm_Horizontal" V 5180 3900 50  0001 C CNN
@@
 AR Path="/5E9DEC5E/5EA649A8" Ref="J22"  Part="1"
 AR Path="/5E9DEC7B/5EA649A8" Ref="J23"  Part="1"
-F 0 "J16" H 3421 3304 50  0000 R CNN
+F 0 "J20" H 3421 3304 50  0000 R CNN
 F 1 "RJ14" H 3421 3395 50  0000 R CNN
 F 2 "Wurth:615004141121" V 3750 3325 50  0001 C CNN
@@
 AR Path="/5E9DEC5E/5EA66D61" Ref="R25"  Part="1"
 AR Path="/5E9DEC7B/5EA66D61" Ref="R27"  Part="1"
-F 0 "R15" H 6220 3946 50  0000 L CNN
+F 0 "R23" H 6220 3946 50  0000 L CNN
 F 1 "220K" H 6220 3855 50  0000 L CNN
 F 2 "Resistor_THT:R_Axial_DIN0207_L6.3mm_D2.5mm_P10.16mm_Horizontal" V 6080 3900 50  0001 C CNN
@@
 AR Path="/5EA83CCC/5E9E2B63" Ref="R30"  Part="1"
 AR Path="/5EA86618/5E9E2B63" Ref="R31"  Part="1"
-F 0 "R27" H 6370 3096 50  0000 L CNN
+F 0 "R31" H 6370 3096 50  0000 L CNN
 F 1 "10K" H 6370 3005 50  0000 L CNN
 F 2 "Resistor_THT:R_Axial_DIN0207_L6.3mm_D2.5mm_P10.16mm_Horizontal" V 6230 3050 50  0001 C CNN

Commit message: Final updates to unified BoB
Parts:
- R14, R15, R27: footprint Resistor_THT:R_Axial_DIN0207_L6.3mm_D2.5mm_P10.16mm_Horizontal -> Resistor_THT:R_Axial_DIN0207_L6.3mm_D2.5mm_P7.62mm_Horizontal
Changed lines of the file:
@@
 AR Path="/5E9DEC5E/5EA62D6B" Ref="U7"  Part="1"
 AR Path="/5E9DEC7B/5EA62D6B" Ref="U8"  Part="1"
-F 0 "U6" H 5750 3825 50  0000 C CNN
+F 0 "U2" H 5750 3825 50  0000 C CNN
 F 1 "4N35" H 5750 3734 50  0000 C CNN
 F 2 "Package_DIP:DIP-6_W7.62mm" H 5550 3300 50  0001 L CIN
@@
 AR Path="/5E9DEC5E/5EA63E66" Ref="R24"  Part="1"
 AR Path="/5E9DEC7B/5EA63E66" Ref="R26"  Part="1"
-F 0 "R22" H 5320 3946 50  0000 L CNN
+F 0 "R14" H 5320 3946 50  0000 L CNN
 F 1 "2K2" H 5320 3855 50  0000 L CNN
-F 2 "Resistor_THT:R_Axial_DIN0207_L6.3mm_D2.5mm_P10.16mm_Horizontal" V 5180 3900 50  0001 C CNN
+F 2 "Resistor_THT:R_Axial_DIN0207_L6.3mm_D2.5mm_P7.62mm_Horizontal" V 5180 3900 50  0001 C CNN
 F 3 "~" H 5250 3900 50  0001 C CNN
 F 4 "CFR-25JB-52-2K2" H 5250 3900 50  0001 C CNN "MPN"
@@
 AR Path="/5E9DEC5E/5EA649A8" Ref="J22"  Part="1"
 AR Path="/5E9DEC7B/5EA649A8" Ref="J23"  Part="1"
-F 0 "J20" H 3421 3304 50  0000 R CNN
+F 0 "J16" H 3421 3304 50  0000 R CNN
 F 1 "RJ14" H 3421 3395 50  0000 R CNN
 F 2 "Wurth:615004141121" V 3750 3325 50  0001 C CNN
@@
 AR Path="/5E9DEC5E/5EA66D61" Ref="R25"  Part="1"
 AR Path="/5E9DEC7B/5EA66D61" Ref="R27"  Part="1"
-F 0 "R23" H 6220 3946 50  0000 L CNN
+F 0 "R15" H 6220 3946 50  0000 L CNN
 F 1 "220K" H 6220 3855 50  0000 L CNN
-F 2 "Resistor_THT:R_Axial_DIN0207_L6.3mm_D2.5mm_P10.16mm_Horizontal" V 6080 3900 50  0001 C CNN
+F 2 "Resistor_THT:R_Axial_DIN0207_L6.3mm_D2.5mm_P7.62mm_Horizontal" V 6080 3900 50  0001 C CNN
 F 3 "~" H 6150 3900 50  0001 C CNN
 F 4 "CFR-25JB-52-220K" H 6150 3900 50  0001 C CNN "MPN"
@@
 AR Path="/5EA83CCC/5E9E2B63" Ref="R30"  Part="1"
 AR Path="/5EA86618/5E9E2B63" Ref="R31"  Part="1"
-F 0 "R31" H 6370 3096 50  0000 L CNN
+F 0 "R27" H 6370 3096 50  0000 L CNN
 F 1 "10K" H 6370 3005 50  0000 L CNN
-F 2 "Resistor_THT:R_Axial_DIN0207_L6.3mm_D2.5mm_P10.16mm_Horizontal" V 6230 3050 50  0001 C CNN
+F 2 "Resistor_THT:R_Axial_DIN0207_L6.3mm_D2.5mm_P7.62mm_Horizontal" V 6230 3050 50  0001 C CNN
 F 3 "~" H 6300 3050 50  0001 C CNN
 F 4 "CFR-25JB-52-10K " H 6300 3050 50  0001 C CNN "MPN"
