File: UnifiedBreakout/UnifiedBreakout/relay.kicad_sch (KiCad schematic)
At the start: 6 parts, among them Q1 BC547

Commit message: WIP updating breakout for electrical enclosure
Parts:
- D5: symbol UnifiedBreakout-rescue:LED-Device -> Device:LED
- D6: symbol UnifiedBreakout-rescue:1N4001-Diode -> Diode:1N4001
- Q1: footprint Package_TO_SOT_THT:TO-92_Inline_Wide -> Package_TO_SOT_THT:TO-92_Inline; symbol UnifiedBreakout-rescue:BC547-Transistor_BJT -> Transistor_BJT:BC547
- R8, R9: symbol UnifiedBreakout-rescue:R-Device -> Device:R
- RL1: symbol UnifiedBreakout-rescue:JW2-Relay -> Relay:JW2; Alternative MPN RTE24012 -> RTE24024; Farnell PN (none) -> 1175021; MPN RT424012 -> RT424024
Connections:
- net +12V renamed +24V
- no-connect marks 0 -> 2
