File: UnifiedBreakout/UnifiedBreakout/UnifiedBreakout.kicad_sch (KiCad schematic)
At the start: 29 parts, among them J6 24V BUS, J7 DRAWBAR+MIST+AXIS_PWR, J8 LIMIT, J9 AUX, U4 G3VM-61A1, U5 G3VM-61A1, U6 G3VM-61A1, U7 4N35

Commit message: Final tweaks for production
Connections:
- no-connect marks 12 -> 16
Other:
- sheet ARGON IO ports: added none; removed PWM_DIR, PWM_SIGNAL, STEPGEN_DIR, STEPGEN_STEP
Changed lines of the file:
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@@
   (junction (at 30.48 63.5) (diameter 0.9144) (color 0 0 0 0)
   )
+  (no_connect (at 85.09 63.5))
   (no_connect (at 210.82 261.62))
   (no_connect (at 133.35 59.69))
   (no_connect (at 85.09 144.78))
+  (no_connect (at 85.09 33.02))
   (no_connect (at 219.71 261.62))
   (no_connect (at 238.76 267.97))
   (no_connect (at 133.35 85.09))
+  (no_connect (at 85.09 60.96))
   (no_connect (at 342.9 231.14))
   (no_connect (at 226.06 261.62))
+  (no_connect (at 85.09 30.48))
   (no_connect (at 342.9 228.6))
   (no_connect (at 133.35 34.29))
@@
     (stroke (width 0) (type solid))
   )
-  (wire (pts (xy 368.3 29.21) (xy 363.22 29.21))
-    (stroke (width 0) (type solid))
-  )
   (wire (pts (xy 81.28 48.26) (xy 130.81 48.26))
     (stroke (width 0) (type solid))
@@
     (stroke (width 0) (type solid))
   )
-  (wire (pts (xy 368.3 36.83) (xy 363.22 36.83))
-    (stroke (width 0) (type solid))
-  )
   (wire (pts (xy 34.29 116.84) (xy 38.1 116.84))
     (stroke (width 0) (type solid))
@@
     (stroke (width 0) (type solid))
   )
-  (wire (pts (xy 363.22 31.75) (xy 368.3 31.75))
-    (stroke (width 0) (type solid))
-  )
   (wire (pts (xy 34.29 35.56) (xy 38.1 35.56))
     (stroke (width 0) (type solid))
@@
   )
   (wire (pts (xy 38.1 40.64) (xy 34.29 40.64))
-    (stroke (width 0) (type solid))
-  )
-  (wire (pts (xy 368.3 39.37) (xy 363.22 39.37))
     (stroke (width 0) (type solid))
   )
@@
     (effects (font (size 1.27 1.27)) (justify right bottom))
   )
-  (label "SPINDLE_STEPGEN_DIR" (at 85.09 63.5 0) (fields_autoplaced)
-    (effects (font (size 1.27 1.27)) (justify left bottom))
-  )
   (label "SPINDLE_ENC_IDX" (at 85.09 73.66 0) (fields_autoplaced)
     (effects (font (size 1.27 1.27)) (justify left bottom))
@@
     (effects (font (size 1.27 1.27)) (justify right bottom))
   )
-  (label "SPINDLE_PWM_SIG" (at 363.22 36.83 180) (fields_autoplaced)
-    (effects (font (size 1.27 1.27)) (justify right bottom))
-  )
   (label "ESTOP" (at 294.64 203.2 180) (fields_autoplaced)
     (effects (font (size 1.27 1.27)) (justify right bottom))
-  )
-  (label "SPINDLE_PWM_DIR" (at 85.09 33.02 0) (fields_autoplaced)
-    (effects (font (size 1.27 1.27)) (justify left bottom))
   )
   (label "PENDANT_SELA" (at 85.09 119.38 0) (fields_autoplaced)
@@
     (effects (font (size 1.27 1.27)) (justify right bottom))
   )
-  (label "SPINDLE_STEPGEN_STEP" (at 85.09 60.96 0) (fields_autoplaced)
-    (effects (font (size 1.27 1.27)) (justify left bottom))
-  )
   (label "PENDANT_SELX" (at 342.9 153.67 180) (fields_autoplaced)
     (effects (font (size 1.27 1.27)) (justify right bottom))
@@
     (effects (font (size 1.27 1.27)) (justify right bottom))
   )
-  (label "SPINDLE_STEPGEN_STEP" (at 363.22 29.21 180) (fields_autoplaced)
-    (effects (font (size 1.27 1.27)) (justify right bottom))
-  )
   (label "PENDANT_ENC_A" (at 85.09 139.7 0) (fields_autoplaced)
     (effects (font (size 1.27 1.27)) (justify left bottom))
@@
     (effects (font (size 1.27 1.27)) (justify right bottom))
   )
-  (label "SPINDLE_PWM_SIG" (at 85.09 30.48 0) (fields_autoplaced)
-    (effects (font (size 1.27 1.27)) (justify left bottom))
-  )
   (label "ALARM" (at 133.35 64.77 180) (fields_autoplaced)
     (effects (font (size 1.27 1.27)) (justify right bottom))
@@
     (effects (font (size 1.27 1.27)) (justify right bottom))
   )
-  (label "SPINDLE_STEPGEN_DIR" (at 363.22 31.75 180) (fields_autoplaced)
-    (effects (font (size 1.27 1.27)) (justify right bottom))
-  )
   (label "PENDANT_MULX10" (at 342.9 176.53 180) (fields_autoplaced)
     (effects (font (size 1.27 1.27)) (justify right bottom))
@@
   )
   (label "PROBE" (at 274.32 106.68 180) (fields_autoplaced)
-    (effects (font (size 1.27 1.27)) (justify right bottom))
-  )
-  (label "SPINDLE_PWM_DIR" (at 363.22 39.37 180) (fields_autoplaced)
     (effects (font (size 1.27 1.27)) (justify right bottom))
   )
@@
       (effects (font (size 1.27 1.27)) (justify left))
     )
-    (pin "STEPGEN_STEP" input (at 368.3 29.21 180)
-      (effects (font (size 1.27 1.27)) (justify left))
-    )
-    (pin "STEPGEN_DIR" input (at 368.3 31.75 180)
-      (effects (font (size 1.27 1.27)) (justify left))
-    )
-    (pin "PWM_SIGNAL" input (at 368.3 36.83 180)
-      (effects (font (size 1.27 1.27)) (justify left))
-    )
-    (pin "PWM_DIR" input (at 368.3 39.37 180)
-      (effects (font (size 1.27 1.27)) (justify left))
-    )
