File: UnifiedBreakout/UnifiedBreakout/argon_estop.kicad_sch (KiCad schematic)
At the start: 1 part, among them J15 ARGON J2.2

Commit message: WIP updating breakout for electrical enclosure
Parts:
- J15: symbol UnifiedBreakout-rescue:RJ45-Connector -> Connector:RJ45
Connections:
- net Gnd renamed GND
- no-connect marks 0 -> 1
Changed lines of the file:
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@@
-(kicad_sch (version 20211123) (generator eeschema)
+(kicad_sch (version 20230121) (generator eeschema)
   (paper "A4")
   (junction (at 109.22 78.74) (diameter 0.9144) (color 0 0 0 0)
   )
+  (no_connect (at 130.81 81.28))
   (wire (pts (xy 130.81 96.52) (xy 109.22 96.52))
-    (stroke (width 0) (type solid) (color 0 0 0 0))
+    (stroke (width 0) (type solid))
   )
   (wire (pts (xy 109.22 78.74) (xy 109.22 67.31))
-    (stroke (width 0) (type solid) (color 0 0 0 0))
+    (stroke (width 0) (type solid))
   )
   (wire (pts (xy 109.22 96.52) (xy 109.22 105.41))
-    (stroke (width 0) (type solid) (color 0 0 0 0))
+    (stroke (width 0) (type solid))
   )
   (wire (pts (xy 109.22 93.98) (xy 109.22 78.74))
-    (stroke (width 0) (type solid) (color 0 0 0 0))
+    (stroke (width 0) (type solid))
   )
   (wire (pts (xy 130.81 93.98) (xy 109.22 93.98))
-    (stroke (width 0) (type solid) (color 0 0 0 0))
+    (stroke (width 0) (type solid))
   )
   (wire (pts (xy 130.81 78.74) (xy 109.22 78.74))
-    (stroke (width 0) (type solid) (color 0 0 0 0))
+    (stroke (width 0) (type solid))
   )
-  (label "ENABLE" (at 113.03 93.98 0)
+  (label "ENABLE" (at 113.03 93.98 0) (fields_autoplaced)
     (effects (font (size 1.27 1.27)) (justify left bottom))
   )
-  (label "STO2" (at 120.65 78.74 0)
+  (label "STO2" (at 120.65 78.74 0) (fields_autoplaced)
     (effects (font (size 1.27 1.27)) (justify left bottom))
   )
-  (hierarchical_label "Gnd" (shape passive) (at 109.22 105.41 270)
+  (hierarchical_label "GND" (shape passive) (at 109.22 105.41 270) (fields_autoplaced)
     (effects (font (size 1.27 1.27)) (justify right))
   )
-  (hierarchical_label "24V" (shape passive) (at 109.22 67.31 90)
+  (hierarchical_label "24V" (shape passive) (at 109.22 67.31 90) (fields_autoplaced)
     (effects (font (size 1.27 1.27)) (justify left))
   )
-  (hierarchical_label "ESTOP+" (shape input) (at 130.81 86.36 180)
+  (hierarchical_label "ESTOP+" (shape input) (at 130.81 86.36 180) (fields_autoplaced)
     (effects (font (size 1.27 1.27)) (justify right))
   )
-  (hierarchical_label "ESTOP-" (shape input) (at 130.81 88.9 180)
+  (hierarchical_label "ESTOP-" (shape input) (at 130.81 88.9 180) (fields_autoplaced)
     (effects (font (size 1.27 1.27)) (justify right))
   )
-  (hierarchical_label "RS485_B" (shape bidirectional) (at 130.81 91.44 180)
+  (hierarchical_label "RS485_B" (shape bidirectional) (at 130.81 91.44 180) (fields_autoplaced)
     (effects (font (size 1.27 1.27)) (justify right))
   )
-  (hierarchical_label "RS485_A" (shape bidirectional) (at 130.81 83.82 180)
+  (hierarchical_label "RS485_A" (shape bidirectional) (at 130.81 83.82 180) (fields_autoplaced)
     (effects (font (size 1.27 1.27)) (justify right))
   )
-  (symbol (lib_id "UnifiedBreakout-rescue:RJ45-Connector") (at 140.97 86.36 180) (unit 1)
-    (in_bom yes) (on_board yes)
-    (property "Reference" "J15" (id 0) (at 149.352 86.4616 0)
+  (symbol (lib_id "Connector:RJ45") (at 140.97 86.36 180) (unit 1)
+    (in_bom yes) (on_board yes) (dnp no)
+    (property "Reference" "J15" (at 149.352 86.4616 0)
       (effects (font (size 1.27 1.27)) (justify right))
     )
-    (property "Value" "ARGON J2.2" (id 1) (at 149.352 88.773 0)
+    (property "Value" "ARGON J2.2" (at 149.352 88.773 0)
       (effects (font (size 1.27 1.27)) (justify right))
     )
-    (property "Footprint" "Stewart:SS6488SANF1" (id 2) (at 140.97 86.995 90)
+    (property "Footprint" "Stewart:SS6488SANF1" (at 140.97 86.995 90)
       (effects (font (size 1.27 1.27)) hide)
     )
-    (property "Datasheet" "~" (id 3) (at 140.97 86.995 90)
+    (property "Datasheet" "~" (at 140.97 86.995 90)
       (effects (font (size 1.27 1.27)) hide)
     )
-    (property "MPN" "SS-6488S-A-NF-1" (id 4) (at 140.97 86.36 0)
+    (property "MPN" "SS-6488S-A-NF-1" (at 140.97 86.36 0)
       (effects (font (size 1.27 1.27)) hide)
     )
-    (property "Manufacturer" "Bel" (id 5) (at 140.97 86.36 0)
+    (property "Manufacturer" "Bel" (at 140.97 86.36 0)
+      (effects (font (size 1.27 1.27)) hide)
+    )
+    (property "Farnell PN" "" (at 140.97 86.36 0)
       (effects (font (size 1.27 1.27)) hide)
     )
@@
     (pin "7")
     (pin "8")
+    (instances
+      (project "UnifiedBreakout"
+        (path "/e63e39d7-6ac0-4ffd-8aa3-1841a4541b55/00000000-0000-0000-0000-00005ea599cb"
+          (reference "J15") (unit 1)
+        )
+      )
+    )
   )
 )

Commit message: Grouped 4 way RJ45s
Parts:
- removed J15: ARGON J2.2, Stewart:SS6488SANF1, symbol Connector:RJ45
- added J8: (no value), UnifiedBreakout:SS71800-041F, symbol UnifiedBreakout:SS71800-041F
Connections:
- net 24V: now also J8.1_4 (P1_4), J8.7_4 (P7_4)
- net ESTOP+: now also J8.4_4 (P4_4)
- net ESTOP-: now also J8.5_4 (P5_4)
- net GND: now also J8.8_4 (P8_4)
- net RS485_A: now also J8.3_4 (P3_4)
- net RS485_B: now also J8.6_4 (P6_4)
Changed lines of the file:
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@@
     (effects (font (size 1.27 1.27)) (justify right))
   )
-  (symbol (lib_id "Connector:RJ45") (at 140.97 86.36 180) (unit 1)
+  (symbol (lib_id "UnifiedBreakout:SS71800-041F") (at 143.51 87.63 0) (mirror y) (unit 4)
     (in_bom yes) (on_board yes) (dnp no)
-    (property "Reference" "J15" (at 149.352 86.4616 0)
+    (property "Reference" "J8" (at 152.4 92.075 0)
       (effects (font (size 1.27 1.27)) (justify right))
     )
-    (property "Value" "ARGON J2.2" (at 149.352 88.773 0)
+    (property "Value" "" (at 152.4 89.535 0)
       (effects (font (size 1.27 1.27)) (justify right))
     )
-    (property "Footprint" "Stewart:SS6488SANF1" (at 140.97 86.995 90)
+    (property "Footprint" "UnifiedBreakout:SS71800-041F" (at 143.51 87.63 0)
+      (effects (font (size 1.27 1.27)) (justify bottom) hide)
+    )
+    (property "Datasheet" "" (at 143.51 87.63 0)
       (effects (font (size 1.27 1.27)) hide)
     )
-    (property "Datasheet" "~" (at 140.97 86.995 90)
-      (effects (font (size 1.27 1.27)) hide)
+    (property "MPN" "SS71800-041F" (at 152.4 86.995 0)
+      (effects (font (size 1.27 1.27)) (justify right) hide)
     )
-    (property "MPN" "SS-6488S-A-NF-1" (at 140.97 86.36 0)
-      (effects (font (size 1.27 1.27)) hide)
+    (property "Manufacturer" "Stewart Connector" (at 152.4 84.455 0)
+      (effects (font (size 1.27 1.27)) (justify right) hide)
     )
-    (property "Manufacturer" "Bel" (at 140.97 86.36 0)
-      (effects (font (size 1.27 1.27)) hide)
+    (property "Farnell PN" "2891045" (at 152.4 81.915 0)
+      (effects (font (size 1.27 1.27)) (justify right) hide)
     )
-    (property "Farnell PN" "" (at 140.97 86.36 0)
-      (effects (font (size 1.27 1.27)) hide)
-    )
-    (pin "1")
-    (pin "2")
-    (pin "3")
-    (pin "4")
-    (pin "5")
-    (pin "6")
-    (pin "7")
-    (pin "8")
+    (pin "1_1")
+    (pin "2_1")
+    (pin "3_1")
+    (pin "4_1")
+    (pin "5_1")
+    (pin "6_1")
+    (pin "7_1")
+    (pin "8_1")
+    (pin "S1")
+    (pin "S2")
+    (pin "S3")
+    (pin "S4")
+    (pin "S5")
+    (pin "1_2")
+    (pin "2_2")
+    (pin "3_2")
+    (pin "4_2")
+    (pin "5_2")
+    (pin "6_2")
+    (pin "7_2")
+    (pin "8_2")
+    (pin "1_3")
+    (pin "2_3")
+    (pin "3_3")
+    (pin "4_3")
+    (pin "5_3")
+    (pin "6_3")
+    (pin "7_3")
+    (pin "8_3")
+    (pin "1_4")
+    (pin "2_4")
+    (pin "3_4")
+    (pin "4_4")
+    (pin "5_4")
+    (pin "6_4")
+    (pin "7_4")
+    (pin "8_4")
     (instances
       (project "UnifiedBreakout"
         (path "/e63e39d7-6ac0-4ffd-8aa3-1841a4541b55/00000000-0000-0000-0000-00005ea599cb"
-          (reference "J15") (unit 1)
+          (reference "J8") (unit 4)
         )
       )

Commit message: Update IO and opto
Parts:
- J3: renamed from J8; value (none) -> ~
Changed lines of the file:
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@@
   (symbol (lib_id "UnifiedBreakout:SS71800-041F") (at 143.51 87.63 0) (mirror y) (unit 4)
     (in_bom yes) (on_board yes) (dnp no)
-    (property "Reference" "J8" (at 152.4 92.075 0)
+    (property "Reference" "J3" (at 152.4 92.075 0)
       (effects (font (size 1.27 1.27)) (justify right))
     )
-    (property "Value" "" (at 152.4 89.535 0)
+    (property "Value" "~" (at 152.4 89.535 0)
       (effects (font (size 1.27 1.27)) (justify right))
     )
@@
       (project "UnifiedBreakout"
         (path "/e63e39d7-6ac0-4ffd-8aa3-1841a4541b55/00000000-0000-0000-0000-00005ea599cb"
-          (reference "J8") (unit 4)
+          (reference "J3") (unit 4)
         )
       )

Commit message: Started some layout
Connections:
- net 24V: now also J3.1_1 (P1_1), J3.7_1 (P7_1); no longer J3.1_4 (P1_4), J3.7_4 (P7_4)
- net ESTOP+: now also J3.4_1 (P4_1); no longer J3.4_4 (P4_4)
- net ESTOP-: now also J3.5_1 (P5_1); no longer J3.5_4 (P5_4)
- net GND: now also J3.8_1 (P8_1); no longer J3.8_4 (P8_4)
- net RS485_A: now also J3.3_1 (P3_1); no longer J3.3_4 (P3_4)
- net RS485_B: now also J3.6_1 (P6_1); no longer J3.6_4 (P6_4)
- new net: J3.S1 (SHIELD), J3.S2 (SHIELD), J3.S3 (SHIELD), J3.S4 (SHIELD), J3.S5 (SHIELD)
Changed lines of the file:
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@@
     (effects (font (size 1.27 1.27)) (justify right))
   )
-  (symbol (lib_id "UnifiedBreakout:SS71800-041F") (at 143.51 87.63 0) (mirror y) (unit 4)
+  (symbol (lib_id "UnifiedBreakout:SS71800-041F") (at 143.51 87.63 0) (mirror y) (unit 1)
     (in_bom yes) (on_board yes) (dnp no)
     (property "Reference" "J3" (at 152.4 92.075 0)
@@
       (project "UnifiedBreakout"
         (path "/e63e39d7-6ac0-4ffd-8aa3-1841a4541b55/00000000-0000-0000-0000-00005ea599cb"
-          (reference "J3") (unit 4)
+          (reference "J3") (unit 1)
         )
       )

Commit message: Some layout
Parts:
- renumbered J3 to J4
Changed lines of the file:
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@@
   (symbol (lib_id "UnifiedBreakout:SS71800-041F") (at 143.51 87.63 0) (mirror y) (unit 1)
     (in_bom yes) (on_board yes) (dnp no)
-    (property "Reference" "J3" (at 152.4 92.075 0)
+    (property "Reference" "J4" (at 152.4 92.075 0)
       (effects (font (size 1.27 1.27)) (justify right))
     )
@@
       (project "UnifiedBreakout"
         (path "/e63e39d7-6ac0-4ffd-8aa3-1841a4541b55/00000000-0000-0000-0000-00005ea599cb"
-          (reference "J3") (unit 1)
+          (reference "J4") (unit 1)
         )
       )
