File: UnifiedBreakout/UnifiedBreakout/argon_estop.kicad_sch (KiCad schematic)
At the start: 1 part

Commit message: v3.1
Changed lines of the file:
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@@
     (pin "7_1")
     (pin "8_1")
-    (pin "S1")
-    (pin "S2")
-    (pin "S3")
-    (pin "S4")
-    (pin "S5")
     (pin "1_2")
     (pin "2_2")
