File: UnifiedBreakout/UnifiedBreakout/jog_pendant.kicad_sch (KiCad schematic)
At the start: 1 part, among them J21 PENDANT

Commit message: WIP updating breakout for electrical enclosure
Parts:
- J21: symbol UnifiedBreakout-rescue:DB25_Female_MountingHoles-Connector -> Connector:DB25_Receptacle_MountingHoles; Farnell PN (none) -> 2059751; MPN ID25S33E4GX00LF -> 5747846-4; Manufacturer Amphenol -> AMP - TE Connectivity
Connections:
- no-connect marks 0 -> 11
Changed lines of the file:
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@@
-(kicad_sch (version 20211123) (generator eeschema)
+(kicad_sch (version 20230121) (generator eeschema)
   (paper "A4")
   (junction (at 88.9 142.24) (diameter 0.9144) (color 0 0 0 0)
@@
   (junction (at 82.55 142.24) (diameter 0.9144) (color 0 0 0 0)
   )
+  (no_connect (at 135.89 80.01))
+  (no_connect (at 135.89 115.57))
+  (no_connect (at 135.89 107.95))
+  (no_connect (at 135.89 85.09))
+  (no_connect (at 135.89 97.79))
+  (no_connect (at 135.89 87.63))
+  (no_connect (at 135.89 102.87))
+  (no_connect (at 135.89 105.41))
+  (no_connect (at 135.89 110.49))
+  (no_connect (at 135.89 123.19))
+  (no_connect (at 135.89 92.71))
   (wire (pts (xy 135.89 69.85) (xy 66.04 69.85))
-    (stroke (width 0) (type solid) (color 0 0 0 0))
+    (stroke (width 0) (type solid))
   )
   (wire (pts (xy 135.89 82.55) (xy 97.79 82.55))
-    (stroke (width 0) (type solid) (color 0 0 0 0))
+    (stroke (width 0) (type solid))
   )
   (wire (pts (xy 102.87 113.03) (xy 135.89 113.03))
-    (stroke (width 0) (type solid) (color 0 0 0 0))
+    (stroke (width 0) (type solid))
   )
   (wire (pts (xy 88.9 142.24) (xy 143.51 142.24))
-    (stroke (width 0) (type solid) (color 0 0 0 0))
+    (stroke (width 0) (type solid))
   )
   (wire (pts (xy 135.89 72.39) (xy 97.79 72.39))
-    (stroke (width 0) (type solid) (color 0 0 0 0))
+    (stroke (width 0) (type solid))
   )
   (wire (pts (xy 88.9 95.25) (xy 88.9 142.24))
-    (stroke (width 0) (type solid) (color 0 0 0 0))
+    (stroke (width 0) (type solid))
   )
   (wire (pts (xy 135.89 118.11) (xy 102.87 118.11))
-    (stroke (width 0) (type solid) (color 0 0 0 0))
+    (stroke (width 0) (type solid))
   )
   (wire (pts (xy 135.89 64.77) (xy 66.04 64.77))
-    (stroke (width 0) (type solid) (color 0 0 0 0))
+    (stroke (width 0) (type solid))
   )
   (wire (pts (xy 82.55 142.24) (xy 82.55 148.59))
-    (stroke (width 0) (type solid) (color 0 0 0 0))
+    (stroke (width 0) (type solid))
   )
   (wire (pts (xy 135.89 62.23) (xy 97.79 62.23))
-    (stroke (width 0) (type solid) (color 0 0 0 0))
+    (stroke (width 0) (type solid))
   )
   (wire (pts (xy 143.51 128.27) (xy 143.51 142.24))
-    (stroke (width 0) (type solid) (color 0 0 0 0))
+    (stroke (width 0) (type solid))
   )
   (wire (pts (xy 54.61 77.47) (xy 135.89 77.47))
-    (stroke (width 0) (type solid) (color 0 0 0 0))
+    (stroke (width 0) (type solid))
   )
   (wire (pts (xy 88.9 142.24) (xy 82.55 142.24))
-    (stroke (width 0) (type solid) (color 0 0 0 0))
+    (stroke (width 0) (type solid))
   )
   (wire (pts (xy 135.89 67.31) (xy 97.79 67.31))
-    (stroke (width 0) (type solid) (color 0 0 0 0))
+    (stroke (width 0) (type solid))
   )
   (wire (pts (xy 86.36 120.65) (xy 86.36 36.83))
-    (stroke (width 0) (type solid) (color 0 0 0 0))
+    (stroke (width 0) (type solid))
   )
   (wire (pts (xy 135.89 120.65) (xy 86.36 120.65))
-    (stroke (width 0) (type solid) (color 0 0 0 0))
+    (stroke (width 0) (type solid))
   )
   (wire (pts (xy 82.55 90.17) (xy 82.55 142.24))
-    (stroke (width 0) (type solid) (color 0 0 0 0))
+    (stroke (width 0) (type solid))
   )
   (wire (pts (xy 135.89 90.17) (xy 82.55 90.17))
-    (stroke (width 0) (type solid) (color 0 0 0 0))
+    (stroke (width 0) (type solid))
   )
   (wire (pts (xy 135.89 74.93) (xy 66.04 74.93))
-    (stroke (width 0) (type solid) (color 0 0 0 0))
+    (stroke (width 0) (type solid))
   )
   (wire (pts (xy 135.89 95.25) (xy 88.9 95.25))
-    (stroke (width 0) (type solid) (color 0 0 0 0))
+    (stroke (width 0) (type solid))
   )
-  (label "ENCODERGND" (at 120.65 95.25 0)
+  (label "ENCODERGND" (at 120.65 95.25 0) (fields_autoplaced)
     (effects (font (size 1.27 1.27)) (justify left bottom))
   )
-  (hierarchical_label "MULX10" (shape output) (at 97.79 72.39 180)
+  (hierarchical_label "MULX10" (shape output) (at 97.79 72.39 180) (fields_autoplaced)
     (effects (font (size 1.27 1.27)) (justify right))
   )
-  (hierarchical_label "ENCODER5V" (shape input) (at 86.36 36.83 90)
+  (hierarchical_label "ENCODER5V" (shape input) (at 86.36 36.83 90) (fields_autoplaced)
     (effects (font (size 1.27 1.27)) (justify left))
   )
-  (hierarchical_label "SELX" (shape output) (at 97.79 62.23 180)
+  (hierarchical_label "SELX" (shape output) (at 97.79 62.23 180) (fields_autoplaced)
     (effects (font (size 1.27 1.27)) (justify right))
   )
-  (hierarchical_label "MULX100" (shape output) (at 66.04 74.93 180)
+  (hierarchical_label "MULX100" (shape output) (at 66.04 74.93 180) (fields_autoplaced)
     (effects (font (size 1.27 1.27)) (justify right))
   )
-  (hierarchical_label "COM" (shape output) (at 82.55 148.59 270)
+  (hierarchical_label "COM" (shape output) (at 82.55 148.59 270) (fields_autoplaced)
     (effects (font (size 1.27 1.27)) (justify right))
   )
-  (hierarchical_label "ENCB" (shape output) (at 102.87 118.11 180)
+  (hierarchical_label "ENCB" (shape output) (at 102.87 118.11 180) (fields_autoplaced)
     (effects (font (size 1.27 1.27)) (justify right))
   )
-  (hierarchical_label "ESTOP-" (shape output) (at 135.89 100.33 180)
+  (hierarchical_label "ESTOP-" (shape output) (at 135.89 100.33 180) (fields_autoplaced)
     (effects (font (size 1.27 1.27)) (justify right))
   )
-  (hierarchical_label "ESTOP+" (shape output) (at 54.61 77.47 180)
+  (hierarchical_label "ESTOP+" (shape output) (at 54.61 77.47 180) (fields_autoplaced)
     (effects (font (size 1.27 1.27)) (justify right))
   )
-  (hierarchical_label "ENCA" (shape output) (at 102.87 113.03 180)
+  (hierarchical_label "ENCA" (shape output) (at 102.87 113.03 180) (fields_autoplaced)
     (effects (font (size 1.27 1.27)) (justify right))
   )
-  (hierarchical_label "SELA" (shape output) (at 97.79 82.55 180)
+  (hierarchical_label "SELA" (shape output) (at 97.79 82.55 180) (fields_autoplaced)
     (effects (font (size 1.27 1.27)) (justify right))
   )
-  (hierarchical_label "MULX1" (shape output) (at 66.04 69.85 180)
+  (hierarchical_label "MULX1" (shape output) (at 66.04 69.85 180) (fields_autoplaced)
     (effects (font (size 1.27 1.27)) (justify right))
   )
-  (hierarchical_label "SELY" (shape output) (at 66.04 64.77 180)
+  (hierarchical_label "SELY" (shape output) (at 66.04 64.77 180) (fields_autoplaced)
     (effects (font (size 1.27 1.27)) (justify right))
   )
-  (hierarchical_label "SELZ" (shape output) (at 97.79 67.31 180)
+  (hierarchical_label "SELZ" (shape output) (at 97.79 67.31 180) (fields_autoplaced)
     (effects (font (size 1.27 1.27)) (justify right))
   )
-  (symbol (lib_id "UnifiedBreakout-rescue:DB25_Female_MountingHoles-Connector") (at 143.51 92.71 0) (unit 1)
-    (in_bom yes) (on_board yes)
-    (property "Reference" "J21" (id 0) (at 148.082 92.6592 0)
+  (symbol (lib_id "Connector:DB25_Receptacle_MountingHoles") (at 143.51 92.71 0) (unit 1)
+    (in_bom yes) (on_board yes) (dnp no)
+    (property "Reference" "J21" (at 148.082 92.6592 0)
       (effects (font (size 1.27 1.27)) (justify left))
     )
-    (property "Value" "PENDANT" (id 1) (at 148.082 94.9706 0)
+    (property "Value" "PENDANT" (at 148.082 94.9706 0)
       (effects (font (size 1.27 1.27)) (justify left))
     )
-    (property "Footprint" "Connector_Dsub:DSUB-25_Female_Horizontal_P2.77x2.84mm_EdgePinOffset7.70mm_Housed_MountingHolesOffset9.12mm" (id 2) (at 143.51 92.71 0)
+    (property "Footprint" "Connector_Dsub:DSUB-25_Female_Horizontal_P2.77x2.84mm_EdgePinOffset7.70mm_Housed_MountingHolesOffset9.12mm" (at 143.51 92.71 0)
       (effects (font (size 1.27 1.27)) hide)
     )
-    (property "Datasheet" " ~" (id 3) (at 143.51 92.71 0)
+    (property "Datasheet" " ~" (at 143.51 92.71 0)
       (effects (font (size 1.27 1.27)) hide)
     )
-    (property "Alternative MPN" "L77SDB25SA4CH4F " (id 4) (at 143.51 92.71 0)
+    (property "Alternative MPN" "L77SDB25SA4CH4F " (at 143.51 92.71 0)
       (effects (font (size 1.27 1.27)) hide)
     )
-    (property "MPN" "ID25S33E4GX00LF" (id 5) (at 143.51 92.71 0)
+    (property "MPN" "5747846-4 " (at 143.51 92.71 0)
       (effects (font (size 1.27 1.27)) hide)
     )
-    (property "Manufacturer" "Amphenol" (id 6) (at 143.51 92.71 0)
+    (property "Manufacturer" "AMP - TE Connectivity" (at 143.51 92.71 0)
+      (effects (font (size 1.27 1.27)) hide)
+    )
+    (property "Farnell PN" "2059751" (at 143.51 92.71 0)
       (effects (font (size 1.27 1.27)) hide)
     )
@@
     (pin "8")
     (pin "9")
+    (instances
+      (project "UnifiedBreakout"
+        (path "/e63e39d7-6ac0-4ffd-8aa3-1841a4541b55/00000000-0000-0000-0000-00005e92536f"
+          (reference "J21") (unit 1)
+        )
+      )
+    )
   )
 )

Commit message: Update IO and opto
Parts:
- renumbered J21 to J4
Changed lines of the file:
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@@
   (symbol (lib_id "Connector:DB25_Receptacle_MountingHoles") (at 143.51 92.71 0) (unit 1)
     (in_bom yes) (on_board yes) (dnp no)
-    (property "Reference" "J21" (at 148.082 92.6592 0)
+    (property "Reference" "J4" (at 148.082 92.6592 0)
       (effects (font (size 1.27 1.27)) (justify left))
     )
@@
       (project "UnifiedBreakout"
         (path "/e63e39d7-6ac0-4ffd-8aa3-1841a4541b55/00000000-0000-0000-0000-00005e92536f"
-          (reference "J21") (unit 1)
+          (reference "J4") (unit 1)
         )
       )

Commit message: Some layout
Parts:
- renumbered J4 to J5
Changed lines of the file:
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@@
   (symbol (lib_id "Connector:DB25_Receptacle_MountingHoles") (at 143.51 92.71 0) (unit 1)
     (in_bom yes) (on_board yes) (dnp no)
-    (property "Reference" "J4" (at 148.082 92.6592 0)
+    (property "Reference" "J5" (at 148.082 92.6592 0)
       (effects (font (size 1.27 1.27)) (justify left))
     )
@@
       (project "UnifiedBreakout"
         (path "/e63e39d7-6ac0-4ffd-8aa3-1841a4541b55/00000000-0000-0000-0000-00005e92536f"
-          (reference "J4") (unit 1)
+          (reference "J5") (unit 1)
         )
       )
