File: UnifiedBreakout/UnifiedBreakout/opto_input.kicad_sch (KiCad schematic)
At the start: 3 parts, among them U1 ILD74

Commit message: V3 BOM
Parts:
- R1: Farnell PN (none) -> 9341536; MPN CFR-25JB-52-2K2 -> MF25 2K2; Manufacturer Yageo -> MULTICOMP PRO
- R2: Farnell PN (none) -> 9341110; MPN CFR-25JB-52-10K -> MF25 10K; Manufacturer Yageo -> MULTICOMP PRO
Changed lines of the file:
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@@
       (effects (font (size 1.27 1.27)) hide)
     )
-    (property "MPN" "CFR-25JB-52-10K " (at 160.02 74.93 0)
+    (property "MPN" "MF25 10K" (at 160.02 74.93 0)
       (effects (font (size 1.27 1.27)) hide)
     )
-    (property "Manufacturer" "Yageo" (at 160.02 74.93 0)
+    (property "Manufacturer" "MULTICOMP PRO" (at 160.02 74.93 0)
       (effects (font (size 1.27 1.27)) hide)
     )
-    (property "Farnell PN" "" (at 160.02 74.93 0)
+    (property "Farnell PN" "9341110" (at 160.02 74.93 0)
       (effects (font (size 1.27 1.27)) hide)
     )
@@
       (effects (font (size 1.27 1.27)) hide)
     )
-    (property "MPN" "CFR-25JB-52-2K2" (at 133.35 99.06 0)
+    (property "MPN" "MF25 2K2" (at 133.35 99.06 0)
       (effects (font (size 1.27 1.27)) hide)
     )
-    (property "Manufacturer" "Yageo" (at 133.35 99.06 0)
+    (property "Manufacturer" "MULTICOMP PRO" (at 133.35 99.06 0)
       (effects (font (size 1.27 1.27)) hide)
     )
-    (property "Farnell PN" "" (at 133.35 99.06 0)
+    (property "Farnell PN" "9341536" (at 133.35 99.06 0)
       (effects (font (size 1.27 1.27)) hide)
     )
