File: control-box-hardware/cnc-interface-panel.kicad_sch (KiCad schematic)
At the start: 52 parts, among them J1 USB_B_Mini, J2 SWD_DAPLINK, J3 3V3-OUT, J4 5V-OUT, J5 GND-OUT, J6 IO-A, J7 IO-B, J8 I2C, SW1 BOOT0, SW2 RESET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

Commit message: Finish laying out CNC encoders PCB
Parts:
- removed H3, H4: ~, MountingHole:MountingHole_3.2mm_M3_Pad_Via, symbol Mechanical:MountingHole_Pad
- removed J6: IO-A, TerminalBlock_Phoenix:TerminalBlock_Phoenix_MKDS-1,5-4_1x04_P5.00mm_Horizontal, symbol Connector:Screw_Terminal_01x04
- removed J7: IO-B, TerminalBlock_Phoenix:TerminalBlock_Phoenix_MKDS-1,5-4_1x04_P5.00mm_Horizontal, symbol Connector:Screw_Terminal_01x04
- J2, J3, J4, J5: now not fitted
- J8, R3, R4: now not fitted; now left out of the parts list
Connections:
- net CASE: no longer H1.1
- net FEED_A: now also U1.30 (PA9); no longer U1.29 (PA8)
- net FEED_B: now also U1.29 (PA8); no longer U1.30 (PA9)
- net GND: no longer U1.7 (NRST)
- net I2C_SCL: now also J8.2 (Pin_2); no longer J8.3 (Pin_3)
- net I2C_SDA: now also J8.3 (Pin_3); no longer J8.2 (Pin_2)
- net RAPID_A: now also U1.17 (PA7); no longer U1.16 (PA6)
- net RAPID_B: now also U1.16 (PA6); no longer U1.17 (PA7)
- net RAPID_RESET: now also U1.18 (PB0); no longer U1.15 (PA5)
- net RST: now also J2.1 (Pin_1); no longer J2.4 (Pin_4)
- net SWD: now also J2.4 (Pin_4); no longer J2.1 (Pin_1)
- net at C3.1, R2.2, SW2.2: now also U1.7 (NRST)
- no-connect marks 14 -> 23

Commit message: Fix control box PCB issues, add USB connector to BOM
Parts:
- removed R5, R6: 560, Resistor_SMD:R_0603_1608Metric_Pad0.98x0.95mm_HandSolder, symbol Device:R_Small
- added R19, R20, R21: 1k5, Resistor_SMD:R_0603_1608Metric_Pad0.98x0.95mm_HandSolder, symbol Device:R_Small
- J1: JLCPCB (none) -> C136451; MPN (none) -> 67503-1020; Manufacturer (none) -> MOLEX; now in the parts list
Connections:
- net +3V3: now also R19.1, R20.2
- net D+: now also R19.2
- net FEED_RESET: no longer C9.1, R8.2
- net LED: now also R21.2
- net RAPID_RESET: no longer C13.1, R18.2
- net at R17.2, SW4.S1: now also C13.1, R18.2
- net at D1.2 (A): now also R20.1
- net at R9.2, SW3.S1: now also C9.1, R8.2
- net at D2.2 (A): now also R21.1
Other:
- moved on the sheet: R17, R9
